File: _autosave-matrix.kicad_sch (KiCad schematic)
At the start: 208 parts, among them SW10 F7, SW100 RCRTL, SW101 arrow_LT, SW102 arrow_DN, SW103 arrow_RT, SW104 num_0, SW105 num_DEL, SW106 num_ENTER, SW11 F8, SW12 F9, SW13 F10, SW14 F11, SW15 F12, SW16 G1, SW17 `, SW18 1, SW19 2, SW20 3, SW21 4, SW22 5, SW23 6, SW24 7, SW25 8, SW26 9, SW27 0, SW28 -, SW29 =, SW3 esc, SW30 Backspace, SW31 insert, SW32 home, SW33 NUM_lock, SW34 num_/, SW35 num_*, SW36 num_-, SW37 G2, SW38 TAB, SW39 Q, SW4 F1, SW40 W, SW41 E, SW42 R, SW43 T, SW44 Y, SW45 U, SW46 I, SW47 O, SW48 P, SW49 [, SW5 F2, SW50 ], SW51 \, SW52 END, SW53 PGUP, SW54 num_7, SW55 num_8, SW56 num_9, SW57 G3, SW58 CAP_LOCK, SW59 A, SW6 F3, SW60 S, SW61 D, SW62 F, SW63 G, SW64 H, SW65 J, SW66 K, SW67 L, SW68 ;, SW69 ', SW7 F4, SW70 ENTER, SW71 DELETE, SW72 PGDN, SW73 num_4, SW74 num_5, SW75 num_6, SW76 num_+, SW77 G4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

Commit message: project resumed
Parts:
- removed D10, D11, D12, D13, D9: D, Diode_SMD:D_SOD-123, symbol Device:D
- removed SW10: F7, Alps_Only:ALPS-1U, symbol Switch:SW_Push
- removed SW11: F8, Alps_Only:ALPS-1U, symbol Switch:SW_Push
- removed SW12: F9, Alps_Only:ALPS-1U, symbol Switch:SW_Push
- removed SW13: F10, Alps_Only:ALPS-1U, symbol Switch:SW_Push
- removed SW14: F11, Alps_Only:ALPS-1U, symbol Switch:SW_Push
- removed SW15: F12, Alps_Only:ALPS-1U, symbol Switch:SW_Push
- removed SW3: esc, Alps_Only:ALPS-1U, symbol Switch:SW_Push
- removed SW4: F1, Alps_Only:ALPS-1U, symbol Switch:SW_Push
- removed SW5: F2, Alps_Only:ALPS-1U, symbol Switch:SW_Push
- removed SW6: F3, Alps_Only:ALPS-1U, symbol Switch:SW_Push
- removed SW7: F4, Alps_Only:ALPS-1U, symbol Switch:SW_Push
- removed SW8: F5, Alps_Only:ALPS-1U, symbol Switch:SW_Push
- removed SW9: F6, Alps_Only:ALPS-1U, symbol Switch:SW_Push
- added MX1, MX2, MX3, MX4, MX5, MX6, MX7, MX8: MX_SW_HS, PCM_marbastlib-mx:SW_MX_HS_CPG151101S11_1u, symbol PCM_marbastlib-mx:MX_SW_HS_CPG151101S11
Connections:
- net col 1: now also MX1.1
- net col 10: now also MX8.1
- net col 2: now also MX2.1
- net col 3: now also MX3.1
- net col 4: now also MX4.1
- net col 7: now also MX5.1
- net col 8: now also MX6.1
- net col 9: now also MX7.1
- net at D2.2 (A): now also MX2.2
- net at D4.2 (A): now also MX4.2
- net at D1.2 (A): now also MX1.2
- net at D3.2 (A): now also MX3.2
- net at D5.2 (A): now also MX5.2
- net at D7.2 (A): now also MX7.2
- net at D6.2 (A): now also MX6.2
- net at D8.2 (A): now also MX8.2
Other:
- moved on the sheet: D1
