File: matrix-no_num.kicad_sch (KiCad schematic)
At the start: 208 parts, among them SW10 F7, SW100 RCRTL, SW101 arrow_LT, SW102 arrow_DN, SW103 arrow_RT, SW104 num_0, SW105 num_DEL, SW106 num_ENTER, SW11 F8, SW12 F9, SW13 F10, SW14 F11, SW15 F12, SW16 G1, SW17 `, SW18 1, SW19 2, SW20 3, SW21 4, SW22 5, SW23 6, SW24 7, SW25 8, SW26 9, SW27 0, SW28 -, SW29 =, SW3 esc, SW30 Backspace, SW31 insert, SW32 home, SW33 NUM_lock, SW34 num_/, SW35 num_*, SW36 num_-, SW37 G2, SW38 TAB, SW39 Q, SW4 F1, SW40 W, SW41 E, SW42 R, SW43 T, SW44 Y, SW45 U, SW46 I, SW47 O, SW48 P, SW49 [, SW5 F2, SW50 ], SW51 \, SW52 END, SW53 PGUP, SW54 num_7, SW55 num_8, SW56 num_9, SW57 G3, SW58 CAP_LOCK, SW59 A, SW6 F3, SW60 S, SW61 D, SW62 F, SW63 G, SW64 H, SW65 J, SW66 K, SW67 L, SW68 ;, SW69 ', SW7 F4, SW70 ENTER, SW71 DELETE, SW72 PGDN, SW73 num_4, SW74 num_5, SW75 num_6, SW76 num_+, SW77 G4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

Commit message: project resumed
Parts:
- removed D102, D103, D104, D31, D33, D34, D36, D52, D53, D54, D56, D71, D72, D73, D74, D76, D89, D90, D91, D99: D, Diode_SMD:D_SOD-123, symbol Device:D
- removed SW101: arrow_LT, Alps_Only:ALPS-1U, symbol Switch:SW_Push
- removed SW104: num_0, Alps_Only:ALPS-2U, symbol Switch:SW_Push
- removed SW105: num_DEL, Alps_Only:ALPS-1U, symbol Switch:SW_Push
- removed SW106: num_ENTER, Alps_Only:ALPS-2U, symbol Switch:SW_Push
- removed SW34: num_/, Alps_Only:ALPS-1U, symbol Switch:SW_Push
- removed SW35: num_*, Alps_Only:ALPS-1U, symbol Switch:SW_Push
- removed SW36: num_-, Alps_Only:ALPS-1U, symbol Switch:SW_Push
- removed SW38: TAB, Alps_Only:ALPS-1.5U, symbol Switch:SW_Push
- removed SW54: num_7, Alps_Only:ALPS-1U, symbol Switch:SW_Push
- removed SW55: num_8, Alps_Only:ALPS-1U, symbol Switch:SW_Push
- removed SW56: num_9, Alps_Only:ALPS-1U, symbol Switch:SW_Push
- removed SW58: CAP_LOCK, Alps_Only:ALPS-1.75U, symbol Switch:SW_Push
- removed SW73: num_4, Alps_Only:ALPS-1U, symbol Switch:SW_Push
- removed SW74: num_5, Alps_Only:ALPS-1U, symbol Switch:SW_Push
- removed SW75: num_6, Alps_Only:ALPS-1U, symbol Switch:SW_Push
- removed SW76: num_+, Alps_Only:ALPS-2U, symbol Switch:SW_Push
- removed SW78: LSHIFT, Alps_Only:ALPS-2.25U, symbol Switch:SW_Push
- removed SW91: num_1, Alps_Only:ALPS-1U, symbol Switch:SW_Push
- removed SW92: num_2, Alps_Only:ALPS-1U, symbol Switch:SW_Push
- removed SW93: num_3, Alps_Only:ALPS-1.25U, symbol Switch:SW_Push
- added D49, D65, D85: D, Diode_SMD:D_0201_0603Metric_Pad0.64x0.40mm_HandSolder, symbol Device:D
- added SW50: CAP_LOCK, symbol Switch:SW_Push
- added SW66: LSHIFT, symbol Switch:SW_Push
- added SW86: arrow_LT, symbol Switch:SW_Push
- D1, D10, D11, D12, D13, D14, D15, D16, D17, D18, D19, D2, D20, D21, D22, D23, D24, D25, D26, D27, D28, D29, D3, D30, D32, D4, D5, D6, D7, D8, D9: footprint Diode_SMD:D_SOD-123 -> Diode_SMD:D_0201_0603Metric_Pad0.64x0.40mm_HandSolder
- D31: renamed from D35; footprint Diode_SMD:D_SOD-123 -> Diode_SMD:D_0201_0603Metric_Pad0.64x0.40mm_HandSolder
- D33: renamed from D37; footprint Diode_SMD:D_SOD-123 -> Diode_SMD:D_0201_0603Metric_Pad0.64x0.40mm_HandSolder
- D34: renamed from D38; footprint Diode_SMD:D_SOD-123 -> Diode_SMD:D_0201_0603Metric_Pad0.64x0.40mm_HandSolder
- D35: renamed from D39; footprint Diode_SMD:D_SOD-123 -> Diode_SMD:D_0201_0603Metric_Pad0.64x0.40mm_HandSolder
- D36: renamed from D40; footprint Diode_SMD:D_SOD-123 -> Diode_SMD:D_0201_0603Metric_Pad0.64x0.40mm_HandSolder
- D37: renamed from D41; footprint Diode_SMD:D_SOD-123 -> Diode_SMD:D_0201_0603Metric_Pad0.64x0.40mm_HandSolder
- D38: renamed from D42; footprint Diode_SMD:D_SOD-123 -> Diode_SMD:D_0201_0603Metric_Pad0.64x0.40mm_HandSolder
- D39: renamed from D43; footprint Diode_SMD:D_SOD-123 -> Diode_SMD:D_0201_0603Metric_Pad0.64x0.40mm_HandSolder
- D40: renamed from D44; footprint Diode_SMD:D_SOD-123 -> Diode_SMD:D_0201_0603Metric_Pad0.64x0.40mm_HandSolder
- D41: renamed from D45; footprint Diode_SMD:D_SOD-123 -> Diode_SMD:D_0201_0603Metric_Pad0.64x0.40mm_HandSolder
- D42: renamed from D46; footprint Diode_SMD:D_SOD-123 -> Diode_SMD:D_0201_0603Metric_Pad0.64x0.40mm_HandSolder
- D43: renamed from D47; footprint Diode_SMD:D_SOD-123 -> Diode_SMD:D_0201_0603Metric_Pad0.64x0.40mm_HandSolder
- D44: renamed from D48; footprint Diode_SMD:D_SOD-123 -> Diode_SMD:D_0201_0603Metric_Pad0.64x0.40mm_HandSolder
- D45: renamed from D49; footprint Diode_SMD:D_SOD-123 -> Diode_SMD:D_0201_0603Metric_Pad0.64x0.40mm_HandSolder
- D46: renamed from D50; footprint Diode_SMD:D_SOD-123 -> Diode_SMD:D_0201_0603Metric_Pad0.64x0.40mm_HandSolder
- D47: renamed from D51; footprint Diode_SMD:D_SOD-123 -> Diode_SMD:D_0201_0603Metric_Pad0.64x0.40mm_HandSolder
- D48: renamed from D55; footprint Diode_SMD:D_SOD-123 -> Diode_SMD:D_0201_0603Metric_Pad0.64x0.40mm_HandSolder
- D50: renamed from D57; footprint Diode_SMD:D_SOD-123 -> Diode_SMD:D_0201_0603Metric_Pad0.64x0.40mm_HandSolder
- D51: renamed from D58; footprint Diode_SMD:D_SOD-123 -> Diode_SMD:D_0201_0603Metric_Pad0.64x0.40mm_HandSolder
- D52: renamed from D59; footprint Diode_SMD:D_SOD-123 -> Diode_SMD:D_0201_0603Metric_Pad0.64x0.40mm_HandSolder
- D53: renamed from D60; footprint Diode_SMD:D_SOD-123 -> Diode_SMD:D_0201_0603Metric_Pad0.64x0.40mm_HandSolder
- D54: renamed from D61; footprint Diode_SMD:D_SOD-123 -> Diode_SMD:D_0201_0603Metric_Pad0.64x0.40mm_HandSolder
- D55: renamed from D62; footprint Diode_SMD:D_SOD-123 -> Diode_SMD:D_0201_0603Metric_Pad0.64x0.40mm_HandSolder
- D56: renamed from D63; footprint Diode_SMD:D_SOD-123 -> Diode_SMD:D_0201_0603Metric_Pad0.64x0.40mm_HandSolder
- D57: renamed from D64; footprint Diode_SMD:D_SOD-123 -> Diode_SMD:D_0201_0603Metric_Pad0.64x0.40mm_HandSolder
- D58: renamed from D65; footprint Diode_SMD:D_SOD-123 -> Diode_SMD:D_0201_0603Metric_Pad0.64x0.40mm_HandSolder
- D59: renamed from D66; footprint Diode_SMD:D_SOD-123 -> Diode_SMD:D_0201_0603Metric_Pad0.64x0.40mm_HandSolder
- D60: renamed from D67; footprint Diode_SMD:D_SOD-123 -> Diode_SMD:D_0201_0603Metric_Pad0.64x0.40mm_HandSolder
- D61: renamed from D68; footprint Diode_SMD:D_SOD-123 -> Diode_SMD:D_0201_0603Metric_Pad0.64x0.40mm_HandSolder
- D62: renamed from D69; footprint Diode_SMD:D_SOD-123 -> Diode_SMD:D_0201_0603Metric_Pad0.64x0.40mm_HandSolder
- D63: renamed from D70; footprint Diode_SMD:D_SOD-123 -> Diode_SMD:D_0201_0603Metric_Pad0.64x0.40mm_HandSolder
- D64: renamed from D75; footprint Diode_SMD:D_SOD-123 -> Diode_SMD:D_0201_0603Metric_Pad0.64x0.40mm_HandSolder
- D66: renamed from D77; footprint Diode_SMD:D_SOD-123 -> Diode_SMD:D_0201_0603Metric_Pad0.64x0.40mm_HandSolder
- D67: renamed from D78; footprint Diode_SMD:D_SOD-123 -> Diode_SMD:D_0201_0603Metric_Pad0.64x0.40mm_HandSolder
- D68: renamed from D79; footprint Diode_SMD:D_SOD-123 -> Diode_SMD:D_0201_0603Metric_Pad0.64x0.40mm_HandSolder
- D69: renamed from D80; footprint Diode_SMD:D_SOD-123 -> Diode_SMD:D_0201_0603Metric_Pad0.64x0.40mm_HandSolder
- D70: renamed from D81; footprint Diode_SMD:D_SOD-123 -> Diode_SMD:D_0201_0603Metric_Pad0.64x0.40mm_HandSolder
- D71: renamed from D82; footprint Diode_SMD:D_SOD-123 -> Diode_SMD:D_0201_0603Metric_Pad0.64x0.40mm_HandSolder
- D72: renamed from D83; footprint Diode_SMD:D_SOD-123 -> Diode_SMD:D_0201_0603Metric_Pad0.64x0.40mm_HandSolder
- D73: renamed from D84; footprint Diode_SMD:D_SOD-123 -> Diode_SMD:D_0201_0603Metric_Pad0.64x0.40mm_HandSolder
- D74: renamed from D85; footprint Diode_SMD:D_SOD-123 -> Diode_SMD:D_0201_0603Metric_Pad0.64x0.40mm_HandSolder
- D75: renamed from D86; footprint Diode_SMD:D_SOD-123 -> Diode_SMD:D_0201_0603Metric_Pad0.64x0.40mm_HandSolder
- D76: renamed from D87; footprint Diode_SMD:D_SOD-123 -> Diode_SMD:D_0201_0603Metric_Pad0.64x0.40mm_HandSolder
- D77: renamed from D88; footprint Diode_SMD:D_SOD-123 -> Diode_SMD:D_0201_0603Metric_Pad0.64x0.40mm_HandSolder
- D78: renamed from D92; footprint Diode_SMD:D_SOD-123 -> Diode_SMD:D_0201_0603Metric_Pad0.64x0.40mm_HandSolder
- D79: renamed from D93; footprint Diode_SMD:D_SOD-123 -> Diode_SMD:D_0201_0603Metric_Pad0.64x0.40mm_HandSolder
- D80: renamed from D94; footprint Diode_SMD:D_SOD-123 -> Diode_SMD:D_0201_0603Metric_Pad0.64x0.40mm_HandSolder
- D81: renamed from D95; footprint Diode_SMD:D_SOD-123 -> Diode_SMD:D_0201_0603Metric_Pad0.64x0.40mm_HandSolder
- D82: renamed from D96; footprint Diode_SMD:D_SOD-123 -> Diode_SMD:D_0201_0603Metric_Pad0.64x0.40mm_HandSolder
- D83: renamed from D97; footprint Diode_SMD:D_SOD-123 -> Diode_SMD:D_0201_0603Metric_Pad0.64x0.40mm_HandSolder
- D84: renamed from D98; footprint Diode_SMD:D_SOD-123 -> Diode_SMD:D_0201_0603Metric_Pad0.64x0.40mm_HandSolder
- D86: renamed from D100; footprint Diode_SMD:D_SOD-123 -> Diode_SMD:D_0201_0603Metric_Pad0.64x0.40mm_HandSolder
- D87: renamed from D101; footprint Diode_SMD:D_SOD-123 -> Diode_SMD:D_0201_0603Metric_Pad0.64x0.40mm_HandSolder
- SW10: renamed from SW11; footprint Alps_Only:ALPS-1U -> (none)
- SW11: renamed from SW12; footprint Alps_Only:ALPS-1U -> (none)
- SW12: renamed from SW13; footprint Alps_Only:ALPS-1U -> (none)
- SW13: renamed from SW14; footprint Alps_Only:ALPS-1U -> (none)
- SW14: renamed from SW15; footprint Alps_Only:ALPS-1U -> (none)
- SW15: renamed from SW16; footprint Alps_Only:ALPS-1U -> (none)
- SW16: renamed from SW17; footprint Alps_Only:ALPS-1.25U -> (none)
- SW17: renamed from SW18; footprint Alps_Only:ALPS-1U -> (none)
- SW18: renamed from SW19; footprint Alps_Only:ALPS-1U -> (none)
- SW19: renamed from SW20; footprint Alps_Only:ALPS-1U -> (none)
- SW2: renamed from SW3; footprint Alps_Only:ALPS-1U -> (none)
- SW20: renamed from SW21; footprint Alps_Only:ALPS-1U -> (none)
- SW21: renamed from SW22; footprint Alps_Only:ALPS-1U -> (none)
- SW22: renamed from SW23; footprint Alps_Only:ALPS-1U -> (none)
- SW23: renamed from SW24; footprint Alps_Only:ALPS-1U -> (none)
- SW24: renamed from SW25; footprint Alps_Only:ALPS-1U -> (none)
- SW25: renamed from SW26; footprint Alps_Only:ALPS-1U -> (none)
- SW26: renamed from SW27; footprint Alps_Only:ALPS-1U -> (none)
- SW27: renamed from SW28; footprint Alps_Only:ALPS-1U -> (none)
- SW28: renamed from SW29; footprint Alps_Only:ALPS-1U -> (none)
- SW29: renamed from SW30; footprint Alps_Only:ALPS-1.75U -> (none)
- SW3: renamed from SW4; footprint Alps_Only:ALPS-1U -> (none)
- SW30: renamed from SW31; footprint Alps_Only:ALPS-1U -> (none)
- SW31: renamed from SW32; footprint Alps_Only:ALPS-1U -> (none)
- SW32: renamed from SW37; footprint Alps_Only:ALPS-1U -> (none)
- SW33: value NUM_lock -> TAB; footprint Alps_Only:ALPS-1U -> (none)
- SW34: renamed from SW39; footprint Alps_Only:ALPS-1U -> (none)
- SW35: renamed from SW40; footprint Alps_Only:ALPS-1U -> (none)
- SW36: renamed from SW41; footprint Alps_Only:ALPS-1U -> (none)
- SW37: renamed from SW42; footprint Alps_Only:ALPS-1U -> (none)
- SW38: renamed from SW43; footprint Alps_Only:ALPS-1U -> (none)
- SW39: renamed from SW44; footprint Alps_Only:ALPS-1U -> (none)
- SW4: renamed from SW5; footprint Alps_Only:ALPS-1U -> (none)
- SW40: renamed from SW45; footprint Alps_Only:ALPS-1U -> (none)
- SW41: renamed from SW46; footprint Alps_Only:ALPS-1U -> (none)
- SW42: renamed from SW47; footprint Alps_Only:ALPS-1U -> (none)
- SW43: renamed from SW48; footprint Alps_Only:ALPS-1U -> (none)
- SW44: renamed from SW49; footprint Alps_Only:ALPS-1U -> (none)
- SW45: renamed from SW50; footprint Alps_Only:ALPS-1U -> (none)
- SW46: renamed from SW51; footprint Alps_Only:ALPS-1.5U -> (none)
- SW47: renamed from SW52; footprint Alps_Only:ALPS-1U -> (none)
- SW48: renamed from SW53; footprint Alps_Only:ALPS-1U -> (none)
- SW49: renamed from SW57; footprint Alps_Only:ALPS-1U -> (none)
- SW5: renamed from SW6; footprint Alps_Only:ALPS-1U -> (none)
- SW51: renamed from SW59; footprint Alps_Only:ALPS-1U -> (none)
- SW52: renamed from SW60; footprint Alps_Only:ALPS-1U -> (none)
- SW53: renamed from SW61; footprint Alps_Only:ALPS-1U -> (none)
- SW54: renamed from SW62; footprint Alps_Only:ALPS-1U -> (none)
- SW55: renamed from SW63; footprint Alps_Only:ALPS-1U -> (none)
- SW56: renamed from SW64; footprint Alps_Only:ALPS-1U -> (none)
- SW57: renamed from SW65; footprint Alps_Only:ALPS-1U -> (none)
- SW58: renamed from SW66; footprint Alps_Only:ALPS-1U -> (none)
- SW59: renamed from SW67; footprint Alps_Only:ALPS-1U -> (none)
- SW6: renamed from SW7; footprint Alps_Only:ALPS-1U -> (none)
- SW60: renamed from SW68; footprint Alps_Only:ALPS-1U -> (none)
- SW61: renamed from SW69; footprint Alps_Only:ALPS-1U -> (none)
- SW62: renamed from SW70; footprint Alps_Only:ALPS-2.25U -> (none)
- SW63: renamed from SW71; footprint Alps_Only:ALPS-1U -> (none)
- SW64: renamed from SW72; footprint Alps_Only:ALPS-1U -> (none)
- SW65: renamed from SW77; footprint Alps_Only:ALPS-1U -> (none)
- SW67: renamed from SW79; footprint Alps_Only:ALPS-1U -> (none)
- SW68: renamed from SW80; footprint Alps_Only:ALPS-1U -> (none)
- SW69: renamed from SW81; footprint Alps_Only:ALPS-1U -> (none)
- SW7: renamed from SW8; footprint Alps_Only:ALPS-1U -> (none)
- SW70: renamed from SW82; footprint Alps_Only:ALPS-1U -> (none)
- SW71: renamed from SW83; footprint Alps_Only:ALPS-1U -> (none)
- SW72: renamed from SW84; footprint Alps_Only:ALPS-1U -> (none)
- SW73: renamed from SW85; footprint Alps_Only:ALPS-1U -> (none)
- SW74: renamed from SW86; footprint Alps_Only:ALPS-1U -> (none)
- SW75: renamed from SW87; footprint Alps_Only:ALPS-1U -> (none)
- SW76: renamed from SW88; footprint Alps_Only:ALPS-1U -> (none)
- SW77: renamed from SW89; footprint Alps_Only:ALPS-2.5U -> (none)
- SW78: renamed from SW90; footprint Alps_Only:ALPS-1U -> (none)
- SW79: renamed from SW94; footprint Alps_Only:ALPS-1.25U -> (none)
- SW8: renamed from SW9; footprint Alps_Only:ALPS-1U -> (none)
- SW80: renamed from SW95; footprint Alps_Only:ALPS-1.25U -> (none)
- SW81: renamed from SW96; footprint Alps_Only:ALPS-1.25U -> (none)
- SW82: renamed from SW97; footprint Alps_Only:ALPS-6.25U -> (none)
- SW83: renamed from SW98; footprint Alps_Only:ALPS-1.25U -> (none)
- SW84: renamed from SW99; footprint Alps_Only:ALPS-1.25U -> (none)
- SW85: renamed from SW100; footprint Alps_Only:ALPS-1.25U -> (none)
- SW87: renamed from SW102; footprint Alps_Only:ALPS-1U -> (none)
- SW88: renamed from SW103; footprint Alps_Only:ALPS-1U -> (none)
- SW9: renamed from SW10; footprint Alps_Only:ALPS-1U -> (none)
Connections:
- net col 15 is gone; now on net 2: SW30.1, SW47.1, SW63.1, SW78.1, SW87.1
- net col 16 is gone; now on net 2: SW31.1, SW48.1, SW64.1, SW88.1
- net 2: now also D1.2 (A), D10.2 (A), D11.2 (A), D12.2 (A), D13.2 (A), D14.2 (A), D15.2 (A), D16.2 (A), D17.2 (A), D18.2 (A), D19.2 (A), D2.2 (A), D20.2 (A), D21.2 (A), D22.2 (A), D23.2 (A), D24.2 (A), D25.2 (A), D26.2 (A), D27.2 (A), D28.2 (A), D29.2 (A), D3.2 (A), D30.2 (A), D31.2 (A), D32.2 (A), D33.2 (A), D34.2 (A), D35.2 (A), D36.2 (A), D37.2 (A), D38.2 (A), D39.2 (A), D4.2 (A), D40.2 (A), D42.2 (A), D43.2 (A), D44.2 (A), D45.2 (A), D46.2 (A), D47.2 (A), D48.2 (A), D5.2 (A), D50.2 (A), D51.2 (A), D52.2 (A), D53.2 (A), D54.2 (A), D55.2 (A), D56.2 (A), D57.2 (A), D58.2 (A), D59.2 (A), D6.2 (A), D60.2 (A), D61.2 (A), D62.2 (A), D63.2 (A), D64.2 (A), D66.2 (A), D67.2 (A), D68.2 (A), D69.2 (A), D7.2 (A), D70.2 (A), D71.2 (A), D72.2 (A), D73.2 (A), D74.2 (A), D75.2 (A), D76.2 (A), D77.2 (A), D78.2 (A), D79.2 (A), D8.2 (A), D80.2 (A), D81.2 (A), D82.2 (A), D83.2 (A), D84.2 (A), D86.2 (A), D87.2 (A), D9.2 (A), SW10.1, SW11.1, SW12.1, SW13.1, SW14.1, SW15.1, SW16.1, SW17.1, SW18.1, SW19.1, SW2.1, SW20.1, SW21.1, SW22.1, SW23.1, SW24.1, SW25.1, SW26.1, SW27.1, SW28.1, SW29.1, SW3.1, SW32.1, SW33.1, SW34.1, SW35.1, SW36.1, SW37.1, SW38.1, SW39.1, SW4.1, SW40.1, SW41.1, SW42.1, SW43.1, SW44.1, SW45.1, SW46.1, SW49.1, SW5.1, SW51.1, SW52.1, SW53.1, SW54.1, SW55.1, SW56.1, SW57.1, SW58.1, SW59.1, SW6.1, SW60.1, SW61.1, SW62.1, SW65.1, SW67.1, SW68.1, SW69.1, SW7.1, SW70.1, SW71.1, SW72.1, SW73.1, SW74.1, SW75.1, SW76.1, SW77.1, SW79.1, SW8.1, SW80.1, SW81.1, SW82.1, SW83.1, SW84.1, SW85.1, SW9.1, D49.2 (A), D65.2 (A), D85.2 (A), SW50.1, SW66.1, SW86.1; no longer SW42.2
- net col 0: now also SW15.2, SW32.2, SW49.2, SW65.2; no longer SW15.1, SW32.1, SW49.1, SW65.1
- net col 1: now also SW16.2, SW2.2, SW33.2, SW79.2, SW50.2, SW66.2; no longer SW16.1, SW2.1, SW79.1
- net col 10: now also SW10.2, SW25.2, SW42.2, SW59.2, SW74.2, SW83.2; no longer SW10.1, SW25.1, SW42.1, SW59.1, SW74.1, SW83.1
- net col 11: now also SW11.2, SW26.2, SW43.2, SW60.2, SW75.2; no longer SW11.1, SW26.1, SW43.1, SW60.1, SW75.1
- net col 12: now also SW12.2, SW27.2, SW44.2, SW61.2, SW76.2, SW84.2; no longer SW12.1, SW27.1, SW44.1, SW61.1, SW76.1, SW84.1
- net col 13: now also SW13.2, SW28.2, SW45.2, SW77.2, SW85.2; no longer SW13.1, SW28.1, SW45.1, SW77.1, SW85.1
- net col 14: now also SW14.2, SW29.2, SW46.2, SW62.2, SW86.2; no longer SW14.1, SW29.1, SW46.1, SW62.1
- net col 17: now also SW30.2, SW47.2, SW63.2, SW78.2, SW87.2; no longer SW33.1
- net col 18: now also SW31.2, SW48.2, SW64.2, SW88.2
- net col 2: now also SW17.2, SW3.2, SW34.2, SW51.2, SW80.2; no longer SW17.1, SW3.1, SW34.1, SW51.1, SW80.1
- net col 3: now also SW18.2, SW35.2, SW4.2, SW52.2, SW67.2, SW81.2; no longer SW18.1, SW35.1, SW4.1, SW52.1, SW67.1, SW81.1
- net col 4: now also SW19.2, SW36.2, SW5.2, SW53.2, SW68.2; no longer SW19.1, SW36.1, SW5.1, SW53.1, SW68.1
- net col 5: now also SW20.2, SW37.2, SW54.2, SW6.2, SW69.2; no longer SW20.1, SW37.1, SW54.1, SW6.1, SW69.1
- net col 6: now also SW21.2, SW38.2, SW55.2, SW70.2; no longer SW21.1, SW38.1, SW55.1, SW70.1
- net col 7: now also SW22.2, SW39.2, SW56.2, SW7.2, SW71.2, SW82.2; no longer SW22.1, SW39.1, SW56.1, SW7.1, SW71.1, SW82.1
- net col 8: now also SW23.2, SW40.2, SW57.2, SW72.2, SW8.2; no longer SW23.1, SW40.1, SW57.1, SW72.1, SW8.1
- net col 9: now also SW24.2, SW41.2, SW58.2, SW73.2, SW9.2; no longer SW24.1, SW41.1, SW58.1, SW73.1, SW9.1
- net row 1: no longer D32.1 (K)
- net row 2: now also D32.1 (K)
- net row 3: now also D49.1 (K)
- net row 4: now also D65.1 (K)
- net row 5: now also D85.1 (K)
