File: test2.kicad_pcb (KiCad board)
At the start: 2 copper layers, 100 x 66.7 mm, 19 parts, among them U1 Arduino_Pro_Micro

Commit message: project resumed
Parts:
- removed S1, S2, S3, S4, S5, S6, S7, S8, S9: Keyswitch, ScottoKeebs_MX:MX_PCB_1.00u
- added C2: 22p, Capacitor_SMD:C_0805_2012Metric_Pad1.18x1.45mm_HandSolder, B.Cu at (214.9, 119.9)
- added C3: 22p, Capacitor_SMD:C_0805_2012Metric_Pad1.18x1.45mm_HandSolder, B.Cu at (214.9, 129.4)
- added C4: 0.1u, Capacitor_SMD:C_0805_2012Metric_Pad1.18x1.45mm_HandSolder, B.Cu at (181.0, 129.4)
- added C5: 0.1u, Capacitor_SMD:C_0805_2012Metric_Pad1.18x1.45mm_HandSolder, B.Cu at (210.3, 116.7)
- added C6: 0.1u, Capacitor_SMD:C_0805_2012Metric_Pad1.18x1.45mm_HandSolder, B.Cu at (181.8, 116.1)
- added C7: 0.1u, Capacitor_SMD:C_0805_2012Metric_Pad1.18x1.45mm_HandSolder, B.Cu at (202.4, 112.7)
- added C8: 10u, Capacitor_SMD:C_0805_2012Metric_Pad1.18x1.45mm_HandSolder, B.Cu at (188.1, 111.9)
- added C9: 1u, Capacitor_SMD:C_0805_2012Metric_Pad1.18x1.45mm_HandSolder, B.Cu at (198.4, 104.5)
- added D10: D, Diode_SMD:D_0201_0603Metric_Pad0.64x0.40mm_HandSolder, B.Cu at (258.8, 29.0)
- added D100: D, Diode_SMD:D_0201_0603Metric_Pad0.64x0.40mm_HandSolder, B.Cu at (349.2, 128.2)
- added D101: D, Diode_SMD:D_0201_0603Metric_Pad0.64x0.40mm_HandSolder, B.Cu at (368.3, 128.2)
- added D102: D, Diode_SMD:D_0201_0603Metric_Pad0.64x0.40mm_HandSolder, B.Cu at (401.6, 128.2)
- added D103: D, Diode_SMD:D_0201_0603Metric_Pad0.64x0.40mm_HandSolder, B.Cu at (430.2, 128.2)
- added D104: D, Diode_SMD:D_0201_0603Metric_Pad0.64x0.40mm_HandSolder, B.Cu at (449.3, 120.3)
- added D105: LED, LED_SMD:LED_0805_2012Metric_Pad1.15x1.40mm_HandSolder, F.Cu at (44.3, 191.3)
- added D106: LED, LED_SMD:LED_0805_2012Metric_Pad1.15x1.40mm_HandSolder, F.Cu at (49.1, 191.3)
- added D107: LED, LED_SMD:LED_0805_2012Metric_Pad1.15x1.40mm_HandSolder, F.Cu at (53.8, 191.3)
- added D108: LED, LED_SMD:LED_0805_2012Metric_Pad1.15x1.40mm_HandSolder, F.Cu at (58.9, 191.3)
- added D109: LED, LED_SMD:LED_0805_2012Metric_Pad1.15x1.40mm_HandSolder, F.Cu at (64.1, 191.3)
- added D11: D, Diode_SMD:D_0201_0603Metric_Pad0.64x0.40mm_HandSolder, B.Cu at (277.8, 29.0)
- added D110: LED, LED_SMD:LED_0805_2012Metric_Pad1.15x1.40mm_HandSolder, F.Cu at (68.8, 191.3)
- added D111: LED, LED_SMD:LED_0805_2012Metric_Pad1.15x1.40mm_HandSolder, F.Cu at (73.6, 191.3)
- added D112: LED, LED_SMD:LED_0805_2012Metric_Pad1.15x1.40mm_HandSolder, F.Cu at (78.3, 191.3)
- added D113: LED, LED_SMD:LED_0805_2012Metric_Pad1.15x1.40mm_HandSolder, F.Cu at (83.1, 191.3)
- added D114: LED, LED_SMD:LED_0805_2012Metric_Pad1.15x1.40mm_HandSolder, F.Cu at (87.9, 191.3)
- added D115: LED, LED_SMD:LED_0805_2012Metric_Pad1.15x1.40mm_HandSolder, F.Cu at (92.6, 191.3)
- added D116: LED, LED_SMD:LED_0805_2012Metric_Pad1.15x1.40mm_HandSolder, F.Cu at (97.4, 191.3)
- added D117: LED, LED_SMD:LED_0805_2012Metric_Pad1.15x1.40mm_HandSolder, F.Cu at (102.2, 191.3)
- added D118: LED, LED_SMD:LED_0805_2012Metric_Pad1.15x1.40mm_HandSolder, F.Cu at (106.6, 191.3)
- added D119: LED, LED_SMD:LED_0805_2012Metric_Pad1.15x1.40mm_HandSolder, F.Cu at (111.7, 191.3)
- added D12: D, Diode_SMD:D_0201_0603Metric_Pad0.64x0.40mm_HandSolder, B.Cu at (296.9, 29.0)
- added D120: LED, LED_SMD:LED_0805_2012Metric_Pad1.15x1.40mm_HandSolder, F.Cu at (116.5, 191.3)
- added D121: LED, LED_SMD:LED_0805_2012Metric_Pad1.15x1.40mm_HandSolder, F.Cu at (121.2, 191.3)
- added D122: LED, LED_SMD:LED_0805_2012Metric_Pad1.15x1.40mm_HandSolder, F.Cu at (126.0, 191.3)
- added D123: LED, LED_SMD:LED_0805_2012Metric_Pad1.15x1.40mm_HandSolder, F.Cu at (130.4, 191.3)
- added D124: LED, LED_SMD:LED_0805_2012Metric_Pad1.15x1.40mm_HandSolder, F.Cu at (135.2, 191.3)
- added D125: LED, LED_SMD:LED_0805_2012Metric_Pad1.15x1.40mm_HandSolder, F.Cu at (140.3, 191.3)
- added D126: LED, LED_SMD:LED_0805_2012Metric_Pad1.15x1.40mm_HandSolder, F.Cu at (145.0, 191.3)
- added D127: LED, LED_SMD:LED_0805_2012Metric_Pad1.15x1.40mm_HandSolder, F.Cu at (149.8, 191.3)
- added D128: LED, LED_SMD:LED_0805_2012Metric_Pad1.15x1.40mm_HandSolder, F.Cu at (154.6, 191.3)
- added D129: LED, LED_SMD:LED_0805_2012Metric_Pad1.15x1.40mm_HandSolder, F.Cu at (159.3, 191.3)
- added D13: D, Diode_SMD:D_0201_0603Metric_Pad0.64x0.40mm_HandSolder, B.Cu at (315.9, 29.0)
- added D130: LED, LED_SMD:LED_0805_2012Metric_Pad1.15x1.40mm_HandSolder, F.Cu at (164.1, 191.3)
- added D131: LED, LED_SMD:LED_0805_2012Metric_Pad1.15x1.40mm_HandSolder, F.Cu at (168.5, 191.3)
- added D132: LED, LED_SMD:LED_0805_2012Metric_Pad1.15x1.40mm_HandSolder, F.Cu at (173.3, 191.3)
- added D133: LED, LED_SMD:LED_0805_2012Metric_Pad1.15x1.40mm_HandSolder, F.Cu at (178.0, 191.0)
- added D134: LED, LED_SMD:LED_0805_2012Metric_Pad1.15x1.40mm_HandSolder, F.Cu at (182.8, 191.3)
- added D135: LED, LED_SMD:LED_0805_2012Metric_Pad1.15x1.40mm_HandSolder, F.Cu at (187.6, 191.3)
- added D136: LED, LED_SMD:LED_0805_2012Metric_Pad1.15x1.40mm_HandSolder, F.Cu at (192.3, 191.3)
- added D137: LED, LED_SMD:LED_0805_2012Metric_Pad1.15x1.40mm_HandSolder, F.Cu at (197.4, 191.3)
- added D138: LED, LED_SMD:LED_0805_2012Metric_Pad1.15x1.40mm_HandSolder, F.Cu at (202.2, 191.3)
- added D139: LED, LED_SMD:LED_0805_2012Metric_Pad1.15x1.40mm_HandSolder, F.Cu at (206.9, 191.3)
- added D14: D, Diode_SMD:D_0201_0603Metric_Pad0.64x0.40mm_HandSolder, B.Cu at (30.2, 52.0)
- added D140: LED, LED_SMD:LED_0805_2012Metric_Pad1.15x1.40mm_HandSolder, F.Cu at (211.7, 191.3)
- added D141: LED, LED_SMD:LED_0805_2012Metric_Pad1.15x1.40mm_HandSolder, F.Cu at (216.5, 191.3)
- added D142: LED, LED_SMD:LED_0805_2012Metric_Pad1.15x1.40mm_HandSolder, F.Cu at (221.2, 191.3)
- added D143: LED, LED_SMD:LED_0805_2012Metric_Pad1.15x1.40mm_HandSolder, F.Cu at (226.0, 191.3)
- added D144: LED, LED_SMD:LED_0805_2012Metric_Pad1.15x1.40mm_HandSolder, F.Cu at (230.4, 191.3)
- added D145: LED, LED_SMD:LED_0805_2012Metric_Pad1.15x1.40mm_HandSolder, F.Cu at (235.5, 191.3)
- added D146: LED, LED_SMD:LED_0805_2012Metric_Pad1.15x1.40mm_HandSolder, F.Cu at (239.9, 191.3)
- added D147: LED, LED_SMD:LED_0805_2012Metric_Pad1.15x1.40mm_HandSolder, F.Cu at (244.7, 191.3)
- added D148: LED, LED_SMD:LED_0805_2012Metric_Pad1.15x1.40mm_HandSolder, F.Cu at (249.5, 191.3)
- added D149: LED, LED_SMD:LED_0805_2012Metric_Pad1.15x1.40mm_HandSolder, F.Cu at (254.2, 191.3)
- added D15: D, Diode_SMD:D_0201_0603Metric_Pad0.64x0.40mm_HandSolder, B.Cu at (56.4, 52.0)
- added D150: LED, LED_SMD:LED_0805_2012Metric_Pad1.15x1.40mm_HandSolder, F.Cu at (259.0, 191.3)
- added D151: LED, LED_SMD:LED_0805_2012Metric_Pad1.15x1.40mm_HandSolder, F.Cu at (263.8, 191.3)
- added D152: LED, LED_SMD:LED_0805_2012Metric_Pad1.15x1.40mm_HandSolder, F.Cu at (268.5, 191.3)
- added D153: LED, LED_SMD:LED_0805_2012Metric_Pad1.15x1.40mm_HandSolder, F.Cu at (273.3, 191.3)
- added D154: LED, LED_SMD:LED_0805_2012Metric_Pad1.15x1.40mm_HandSolder, F.Cu at (278.0, 191.3)
- added D155: LED, LED_SMD:LED_0805_2012Metric_Pad1.15x1.40mm_HandSolder, F.Cu at (282.8, 191.3)
- added D156: LED, LED_SMD:LED_0805_2012Metric_Pad1.15x1.40mm_HandSolder, F.Cu at (287.6, 191.3)
- added D157: LED, LED_SMD:LED_0805_2012Metric_Pad1.15x1.40mm_HandSolder, F.Cu at (292.3, 191.3)
- added D158: LED, LED_SMD:LED_0805_2012Metric_Pad1.15x1.40mm_HandSolder, F.Cu at (297.1, 191.3)
- added D159: LED, LED_SMD:LED_0805_2012Metric_Pad1.15x1.40mm_HandSolder, F.Cu at (301.9, 191.3)
- added D16: D, Diode_SMD:D_0201_0603Metric_Pad0.64x0.40mm_HandSolder, B.Cu at (77.8, 52.0)
- added D160: LED, LED_SMD:LED_0805_2012Metric_Pad1.15x1.40mm_HandSolder, F.Cu at (306.6, 191.3)
- added D161: LED, LED_SMD:LED_0805_2012Metric_Pad1.15x1.40mm_HandSolder, F.Cu at (311.4, 191.3)
- added D162: LED, LED_SMD:LED_0805_2012Metric_Pad1.15x1.40mm_HandSolder, F.Cu at (316.1, 191.3)
- added D163: LED, LED_SMD:LED_0805_2012Metric_Pad1.15x1.40mm_HandSolder, F.Cu at (320.9, 191.3)
- added D164: LED, LED_SMD:LED_0805_2012Metric_Pad1.15x1.40mm_HandSolder, F.Cu at (325.7, 191.3)
- added D165: LED, LED_SMD:LED_0805_2012Metric_Pad1.15x1.40mm_HandSolder, F.Cu at (330.4, 191.3)
- added D166: LED, LED_SMD:LED_0805_2012Metric_Pad1.15x1.40mm_HandSolder, F.Cu at (335.2, 191.3)
- added D167: LED, LED_SMD:LED_0805_2012Metric_Pad1.15x1.40mm_HandSolder, F.Cu at (340.0, 191.3)
- added D168: LED, LED_SMD:LED_0805_2012Metric_Pad1.15x1.40mm_HandSolder, F.Cu at (344.7, 191.3)
- added D169: LED, LED_SMD:LED_0805_2012Metric_Pad1.15x1.40mm_HandSolder, F.Cu at (349.5, 191.3)
- added D17: D, Diode_SMD:D_0201_0603Metric_Pad0.64x0.40mm_HandSolder, B.Cu at (96.8, 52.0)
- added D170: LED, LED_SMD:LED_0805_2012Metric_Pad1.15x1.40mm_HandSolder, F.Cu at (354.2, 191.3)
- added D171: LED, LED_SMD:LED_0805_2012Metric_Pad1.15x1.40mm_HandSolder, F.Cu at (359.0, 191.3)
- added D172: LED, LED_SMD:LED_0805_2012Metric_Pad1.15x1.40mm_HandSolder, F.Cu at (364.1, 191.3)
- added D173: LED, LED_SMD:LED_0805_2012Metric_Pad1.15x1.40mm_HandSolder, F.Cu at (368.5, 191.3)
- added D174: LED, LED_SMD:LED_0805_2012Metric_Pad1.15x1.40mm_HandSolder, F.Cu at (373.3, 191.3)
- added D175: LED, LED_SMD:LED_0805_2012Metric_Pad1.15x1.40mm_HandSolder, F.Cu at (378.4, 191.3)
- added D176: LED, LED_SMD:LED_0805_2012Metric_Pad1.15x1.40mm_HandSolder, F.Cu at (383.1, 191.3)
- added D177: LED, LED_SMD:LED_0805_2012Metric_Pad1.15x1.40mm_HandSolder, F.Cu at (387.6, 191.3)
- added D178: LED, LED_SMD:LED_0805_2012Metric_Pad1.15x1.40mm_HandSolder, F.Cu at (392.3, 191.3)
- added D179: LED, LED_SMD:LED_0805_2012Metric_Pad1.15x1.40mm_HandSolder, F.Cu at (397.1, 191.3)
- added D18: D, Diode_SMD:D_0201_0603Metric_Pad0.64x0.40mm_HandSolder, B.Cu at (115.9, 52.0)
- added D180: LED, LED_SMD:LED_0805_2012Metric_Pad1.15x1.40mm_HandSolder, F.Cu at (401.9, 191.3)
- added D181: LED, LED_SMD:LED_0805_2012Metric_Pad1.15x1.40mm_HandSolder, F.Cu at (44.7, 205.6)
- added D182: LED, LED_SMD:LED_0805_2012Metric_Pad1.15x1.40mm_HandSolder, F.Cu at (49.4, 205.6)
- added D183: LED, LED_SMD:LED_0805_2012Metric_Pad1.15x1.40mm_HandSolder, F.Cu at (54.2, 205.6)
- added D184: LED, LED_SMD:LED_0805_2012Metric_Pad1.15x1.40mm_HandSolder, F.Cu at (59.0, 205.6)
- added D185: LED, LED_SMD:LED_0805_2012Metric_Pad1.15x1.40mm_HandSolder, F.Cu at (64.1, 205.6)
- added D186: LED, LED_SMD:LED_0805_2012Metric_Pad1.15x1.40mm_HandSolder, F.Cu at (68.8, 205.6)
- added D187: LED, LED_SMD:LED_0805_2012Metric_Pad1.15x1.40mm_HandSolder, F.Cu at (73.6, 205.6)
- added D188: LED, LED_SMD:LED_0805_2012Metric_Pad1.15x1.40mm_HandSolder, F.Cu at (78.0, 205.6)
- added D189: LED, LED_SMD:LED_0805_2012Metric_Pad1.15x1.40mm_HandSolder, F.Cu at (82.8, 205.6)
- added D19: D, Diode_SMD:D_0201_0603Metric_Pad0.64x0.40mm_HandSolder, B.Cu at (134.9, 52.0)
- added D190: LED, LED_SMD:LED_0805_2012Metric_Pad1.15x1.40mm_HandSolder, F.Cu at (87.5, 205.6)
- added D191: LED, LED_SMD:LED_0805_2012Metric_Pad1.15x1.40mm_HandSolder, F.Cu at (92.3, 205.6)
- added D192: LED, LED_SMD:LED_0805_2012Metric_Pad1.15x1.40mm_HandSolder, F.Cu at (97.1, 205.6)
- added D193: LED, LED_SMD:LED_0805_2012Metric_Pad1.15x1.40mm_HandSolder, F.Cu at (101.8, 205.6)
- added D194: LED, LED_SMD:LED_0805_2012Metric_Pad1.15x1.40mm_HandSolder, F.Cu at (106.6, 205.6)
- added D195: LED, LED_SMD:LED_0805_2012Metric_Pad1.15x1.40mm_HandSolder, F.Cu at (111.4, 205.6)
- added D196: LED, LED_SMD:LED_0805_2012Metric_Pad1.15x1.40mm_HandSolder, F.Cu at (116.5, 205.6)
- added D197: LED, LED_SMD:LED_0805_2012Metric_Pad1.15x1.40mm_HandSolder, F.Cu at (120.9, 205.6)
- added D198: LED, LED_SMD:LED_0805_2012Metric_Pad1.15x1.40mm_HandSolder, F.Cu at (125.6, 205.6)
- added D199: LED, LED_SMD:LED_0805_2012Metric_Pad1.15x1.40mm_HandSolder, F.Cu at (130.4, 205.6)
- added D20: D, Diode_SMD:D_0201_0603Metric_Pad0.64x0.40mm_HandSolder, B.Cu at (154.0, 52.0)
- added D200: LED, LED_SMD:LED_0805_2012Metric_Pad1.15x1.40mm_HandSolder, F.Cu at (135.2, 205.6)
- added D201: LED, LED_SMD:LED_0805_2012Metric_Pad1.15x1.40mm_HandSolder, F.Cu at (139.9, 205.6)
- added D202: LED, LED_SMD:LED_0805_2012Metric_Pad1.15x1.40mm_HandSolder, F.Cu at (145.0, 205.6)
- added D203: LED, LED_SMD:LED_0805_2012Metric_Pad1.15x1.40mm_HandSolder, F.Cu at (149.5, 205.6)
- added D204: LED, LED_SMD:LED_0805_2012Metric_Pad1.15x1.40mm_HandSolder, F.Cu at (154.2, 205.6)
- added D205: LED, LED_SMD:LED_0805_2012Metric_Pad1.15x1.40mm_HandSolder, F.Cu at (159.0, 205.6)
- added D206: LED, LED_SMD:LED_0805_2012Metric_Pad1.15x1.40mm_HandSolder, F.Cu at (163.7, 205.6)
- added D207: LED, LED_SMD:LED_0805_2012Metric_Pad1.15x1.40mm_HandSolder, F.Cu at (168.5, 205.6)
- added D208: LED, LED_SMD:LED_0805_2012Metric_Pad1.15x1.40mm_HandSolder, F.Cu at (173.3, 205.6)
- added D209: LED, LED_SMD:LED_0805_2012Metric_Pad1.15x1.40mm_HandSolder, F.Cu at (178.0, 205.6)
- added D21: D, Diode_SMD:D_0201_0603Metric_Pad0.64x0.40mm_HandSolder, B.Cu at (173.0, 52.0)
- added D22: D, Diode_SMD:D_0201_0603Metric_Pad0.64x0.40mm_HandSolder, B.Cu at (192.1, 52.0)
- added D23: D, Diode_SMD:D_0201_0603Metric_Pad0.64x0.40mm_HandSolder, B.Cu at (211.1, 52.0)
- added D24: D, Diode_SMD:D_0201_0603Metric_Pad0.64x0.40mm_HandSolder, B.Cu at (230.2, 52.0)
- added D25: D, Diode_SMD:D_0201_0603Metric_Pad0.64x0.40mm_HandSolder, B.Cu at (249.2, 52.0)
- added D26: D, Diode_SMD:D_0201_0603Metric_Pad0.64x0.40mm_HandSolder, B.Cu at (268.3, 52.0)
- added D27: D, Diode_SMD:D_0201_0603Metric_Pad0.64x0.40mm_HandSolder, B.Cu at (287.3, 52.8)
- added D28: D, Diode_SMD:D_0201_0603Metric_Pad0.64x0.40mm_HandSolder, B.Cu at (313.5, 52.0)
- added D29: D, Diode_SMD:D_0201_0603Metric_Pad0.64x0.40mm_HandSolder, B.Cu at (346.9, 42.4)
- added D30: D, Diode_SMD:D_0201_0603Metric_Pad0.64x0.40mm_HandSolder, B.Cu at (365.9, 42.5)
- added D31: D, Diode_SMD:D_0201_0603Metric_Pad0.64x0.40mm_HandSolder, B.Cu at (392.1, 52.8)
- added D32: D, Diode_SMD:D_0201_0603Metric_Pad0.64x0.40mm_HandSolder, B.Cu at (411.2, 52.8)
- added D33: D, Diode_SMD:D_0201_0603Metric_Pad0.64x0.40mm_HandSolder, B.Cu at (430.2, 52.8)
- added D34: D, Diode_SMD:D_0201_0603Metric_Pad0.64x0.40mm_HandSolder, B.Cu at (449.3, 52.8)
- added D35: D, Diode_SMD:D_0201_0603Metric_Pad0.64x0.40mm_HandSolder, B.Cu at (30.2, 71.0)
- added D36: D, Diode_SMD:D_0201_0603Metric_Pad0.64x0.40mm_HandSolder, B.Cu at (58.7, 71.1)
- added D37: D, Diode_SMD:D_0201_0603Metric_Pad0.64x0.40mm_HandSolder, B.Cu at (82.5, 71.0)
- added D38: D, Diode_SMD:D_0201_0603Metric_Pad0.64x0.40mm_HandSolder, B.Cu at (101.6, 71.0)
- added D39: D, Diode_SMD:D_0201_0603Metric_Pad0.64x0.40mm_HandSolder, B.Cu at (120.7, 71.1)
- added D40: D, Diode_SMD:D_0201_0603Metric_Pad0.64x0.40mm_HandSolder, B.Cu at (139.7, 71.4)
- added D41: D, Diode_SMD:D_0201_0603Metric_Pad0.64x0.40mm_HandSolder, B.Cu at (158.8, 71.0)
- added D42: D, Diode_SMD:D_0201_0603Metric_Pad0.64x0.40mm_HandSolder, B.Cu at (177.8, 71.0)
- added D43: D, Diode_SMD:D_0201_0603Metric_Pad0.64x0.40mm_HandSolder, B.Cu at (196.8, 71.0)
- added D44: D, Diode_SMD:D_0201_0603Metric_Pad0.64x0.40mm_HandSolder, B.Cu at (215.9, 71.0)
- added D45: D, Diode_SMD:D_0201_0603Metric_Pad0.64x0.40mm_HandSolder, B.Cu at (234.9, 71.0)
- added D46: D, Diode_SMD:D_0201_0603Metric_Pad0.64x0.40mm_HandSolder, B.Cu at (254.0, 71.0)
- added D47: D, Diode_SMD:D_0201_0603Metric_Pad0.64x0.40mm_HandSolder, B.Cu at (273.1, 71.4)
- added D48: D, Diode_SMD:D_0201_0603Metric_Pad0.64x0.40mm_HandSolder, B.Cu at (292.1, 71.4)
- added D49: D, Diode_SMD:D_0201_0603Metric_Pad0.64x0.40mm_HandSolder, B.Cu at (315.9, 71.4)
- added D50: D, Diode_SMD:D_0201_0603Metric_Pad0.64x0.40mm_HandSolder, B.Cu at (346.9, 61.9)
- added D51: D, Diode_SMD:D_0201_0603Metric_Pad0.64x0.40mm_HandSolder, B.Cu at (365.9, 61.6)
- added D52: D, Diode_SMD:D_0201_0603Metric_Pad0.64x0.40mm_HandSolder, B.Cu at (392.1, 71.1)
- added D53: D, Diode_SMD:D_0201_0603Metric_Pad0.64x0.40mm_HandSolder, B.Cu at (411.2, 71.4)
- added D54: D, Diode_SMD:D_0201_0603Metric_Pad0.64x0.40mm_HandSolder, B.Cu at (430.2, 71.4)
- added D55: D, Diode_SMD:D_0201_0603Metric_Pad0.64x0.40mm_HandSolder, B.Cu at (30.2, 90.1)
- added D56: D, Diode_SMD:D_0201_0603Metric_Pad0.64x0.40mm_HandSolder, B.Cu at (61.1, 90.1)
- added D57: D, Diode_SMD:D_0201_0603Metric_Pad0.64x0.40mm_HandSolder, B.Cu at (87.3, 90.1)
- added D58: D, Diode_SMD:D_0201_0603Metric_Pad0.64x0.40mm_HandSolder, B.Cu at (106.4, 90.1)
- added D59: D, Diode_SMD:D_0201_0603Metric_Pad0.64x0.40mm_HandSolder, B.Cu at (125.4, 90.1)
- added D60: D, Diode_SMD:D_0201_0603Metric_Pad0.64x0.40mm_HandSolder, B.Cu at (144.5, 90.1)
- added D61: D, Diode_SMD:D_0201_0603Metric_Pad0.64x0.40mm_HandSolder, B.Cu at (163.5, 90.1)
- added D62: D, Diode_SMD:D_0201_0603Metric_Pad0.64x0.40mm_HandSolder, B.Cu at (182.6, 90.1)
- added D63: D, Diode_SMD:D_0201_0603Metric_Pad0.64x0.40mm_HandSolder, B.Cu at (201.6, 90.1)
- added D64: D, Diode_SMD:D_0201_0603Metric_Pad0.64x0.40mm_HandSolder, B.Cu at (220.7, 90.1)
- added D65: D, Diode_SMD:D_0201_0603Metric_Pad0.64x0.40mm_HandSolder, B.Cu at (239.7, 90.1)
- added D66: D, Diode_SMD:D_0201_0603Metric_Pad0.64x0.40mm_HandSolder, B.Cu at (258.8, 90.1)
- added D67: D, Diode_SMD:D_0201_0603Metric_Pad0.64x0.40mm_HandSolder, B.Cu at (277.8, 90.1)
- added D68: D, Diode_SMD:D_0201_0603Metric_Pad0.64x0.40mm_HandSolder, B.Cu at (308.8, 90.1)
- added D69: D, Diode_SMD:D_0201_0603Metric_Pad0.64x0.40mm_HandSolder, B.Cu at (346.9, 81.0)
- added D70: D, Diode_SMD:D_0201_0603Metric_Pad0.64x0.40mm_HandSolder, B.Cu at (365.9, 80.5)
- added D71: D, Diode_SMD:D_0201_0603Metric_Pad0.64x0.40mm_HandSolder, B.Cu at (392.1, 90.5)
- added D72: D, Diode_SMD:D_0201_0603Metric_Pad0.64x0.40mm_HandSolder, B.Cu at (411.2, 90.8)
- added D73: D, Diode_SMD:D_0201_0603Metric_Pad0.64x0.40mm_HandSolder, B.Cu at (430.2, 90.5)
- added D74: D, Diode_SMD:D_0201_0603Metric_Pad0.64x0.40mm_HandSolder, B.Cu at (449.3, 81.3)
- added D75: D, Diode_SMD:D_0201_0603Metric_Pad0.64x0.40mm_HandSolder, B.Cu at (30.3, 110.0)
- added D76: D, Diode_SMD:D_0201_0603Metric_Pad0.64x0.40mm_HandSolder, B.Cu at (65.9, 109.5)
- added D77: D, Diode_SMD:D_0201_0603Metric_Pad0.64x0.40mm_HandSolder, B.Cu at (96.8, 109.5)
- added D78: D, Diode_SMD:D_0201_0603Metric_Pad0.64x0.40mm_HandSolder, B.Cu at (115.9, 109.9)
- added D79: D, Diode_SMD:D_0201_0603Metric_Pad0.64x0.40mm_HandSolder, B.Cu at (134.9, 109.2)
- added D80: D, Diode_SMD:D_0201_0603Metric_Pad0.64x0.40mm_HandSolder, B.Cu at (154.0, 109.1)
- added D81: D, Diode_SMD:D_0201_0603Metric_Pad0.64x0.40mm_HandSolder, B.Cu at (173.0, 109.2)
- added D82: D, Diode_SMD:D_0201_0603Metric_Pad0.64x0.40mm_HandSolder, B.Cu at (190.5, 109.9)
- added D83: D, Diode_SMD:D_0201_0603Metric_Pad0.64x0.40mm_HandSolder, B.Cu at (211.1, 109.1)
- added D84: D, Diode_SMD:D_0201_0603Metric_Pad0.64x0.40mm_HandSolder, B.Cu at (230.2, 109.1)
- added D85: D, Diode_SMD:D_0201_0603Metric_Pad0.64x0.40mm_HandSolder, B.Cu at (249.2, 109.1)
- added D86: D, Diode_SMD:D_0201_0603Metric_Pad0.64x0.40mm_HandSolder, B.Cu at (268.3, 109.2)
- added D87: D, Diode_SMD:D_0201_0603Metric_Pad0.64x0.40mm_HandSolder, B.Cu at (301.6, 109.1)
- added D88: D, Diode_SMD:D_0201_0603Metric_Pad0.64x0.40mm_HandSolder, B.Cu at (349.2, 109.1)
- added D89: D, Diode_SMD:D_0201_0603Metric_Pad0.64x0.40mm_HandSolder, B.Cu at (392.1, 109.1)
- added D90: D, Diode_SMD:D_0201_0603Metric_Pad0.64x0.40mm_HandSolder, B.Cu at (411.2, 109.1)
- added D91: D, Diode_SMD:D_0201_0603Metric_Pad0.64x0.40mm_HandSolder, B.Cu at (430.2, 109.1)
- added D92: D, Diode_SMD:D_0201_0603Metric_Pad0.64x0.40mm_HandSolder, B.Cu at (56.4, 128.2)
- added D93: D, Diode_SMD:D_0201_0603Metric_Pad0.64x0.40mm_HandSolder, B.Cu at (80.2, 128.2)
- added D94: D, Diode_SMD:D_0201_0603Metric_Pad0.64x0.40mm_HandSolder, B.Cu at (104.0, 128.2)
- added D95: D, Diode_SMD:D_0201_0603Metric_Pad0.64x0.40mm_HandSolder, B.Cu at (175.4, 128.2)
- added D96: D, Diode_SMD:D_0201_0603Metric_Pad0.64x0.40mm_HandSolder, B.Cu at (246.9, 128.2)
- added D97: D, Diode_SMD:D_0201_0603Metric_Pad0.64x0.40mm_HandSolder, B.Cu at (270.7, 128.2)
- added D98: D, Diode_SMD:D_0201_0603Metric_Pad0.64x0.40mm_HandSolder, B.Cu at (294.5, 128.2)
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Connections:
- D1 pad 1: row0 -> row 0
- D2 pad 1: row0 -> row 0
- D3 pad 1: row0 -> row 0
- D4 pad 1: row1 -> row 0
- D5 pad 1: row1 -> row 0
- D6 pad 1: row1 -> row 0
- D7 pad 1: row2 -> row 0
- D8 pad 1: row2 -> row 0
- D9 pad 1: row2 -> row 0
- U1 pad 1: unconnected-(U1-TX0/PD3-Pad1) -> GND
- U1 pad 2: unconnected-(U1-RX1/PD2-Pad2) -> Net-(U1-IO1)
- U1 pad 3: unconnected-(U1-GND-Pad3) -> Net-(U1-IO2)
Routing:
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- removed copper zone on B.Cu, net (none)
- removed copper zone on F.Cu, net (none)
Other:
- board size 100 x 66.7 mm -> 438.2 x 123 mm

Commit message: Finalization of 89 key
Changed 104 keys to 89, removed LEDs, created files needed for production.
Parts:
- removed D100, D101, D102, D103, D104, D88, D89, D90, D91, D92, D93, D94, D95, D96, D97, D98, D99: D, Diode_SMD:D_0201_0603Metric_Pad0.64x0.40mm_HandSolder
- removed D105, D106, D107, D108, D109, D110, D111, D112, D113, D114, D115, D116, D117, D118, D119, D120, D121, D122, D123, D124, D125, D126, D127, D128, D129, D130, D131, D132, D133, D134, D135, D136, D137, D138, D139, D140, D141, D142, D143, D144, D145, D146, D147, D148, D149, D150, D151, D152, D153, D154, D155, D156, D157, D158, D159, D160, D161, D162, D163, D164, D165, D166, D167, D168, D169, D170, D171, D172, D173, D174, D175, D176, D177, D178, D179, D180, D181, D182, D183, D184, D185, D186, D187, D188, D189, D190, D191, D192, D193, D194, D195, D196, D197, D198, D199, D200, D201, D202, D203, D204, D205, D206, D207, D208, D209: LED, LED_SMD:LED_0805_2012Metric_Pad1.15x1.40mm_HandSolder
- removed Q1: BC337, Package_TO_SOT_THT:TO-92_Inline
- removed R10, R100, R101, R102, R103, R104, R105, R106, R107, R108, R109, R11, R110, R111, R112, R113, R12, R13, R14, R15, R16, R17, R18, R19, R20, R21, R22, R23, R24, R25, R26, R27, R28, R29, R30, R31, R32, R33, R34, R35, R36, R37, R38, R39, R40, R41, R42, R43, R44, R45, R46, R47, R48, R49, R50, R51, R52, R53, R54, R55, R56, R57, R58, R59, R60, R61, R62, R63, R64, R65, R66, R67, R68, R69, R70, R71, R72, R73, R74, R75, R76, R77, R78, R79, R80, R81, R82, R83, R84, R85, R86, R87, R88, R89, R90, R91, R92, R93, R94, R95, R96, R97, R98, R99: 1k, Resistor_SMD:R_0805_2012Metric_Pad1.20x1.40mm_HandSolder
- removed SW10: F8, Alps_Only:ALPS-1U
- removed SW100: arrow_LT, Alps_Only:ALPS-1U
- removed SW101: arrow_DN, Alps_Only:ALPS-1U
- removed SW102: arrow_RT, Alps_Only:ALPS-1U
- removed SW103: num_0, Alps_Only:ALPS-2U
- removed SW104: num_DEL, Alps_Only:ALPS-1U
- removed SW105: num_ENTER, Alps_Only:ALPS-2U
- removed SW11: F9, Alps_Only:ALPS-1U
- removed SW12: F10, Alps_Only:ALPS-1U
- removed SW13: F11, Alps_Only:ALPS-1U
- removed SW14: F12, Alps_Only:ALPS-1U
- removed SW15: G1, Alps_Only:ALPS-1U
- removed SW16: `, Alps_Only:ALPS-1.25U
- removed SW17: 1, Alps_Only:ALPS-1U
- removed SW18: 2, Alps_Only:ALPS-1U
- removed SW19: 3, Alps_Only:ALPS-1U
- removed SW20: 4, Alps_Only:ALPS-1U
- removed SW21: 5, Alps_Only:ALPS-1U
- removed SW22: 6, Alps_Only:ALPS-1U
- removed SW23: 7, Alps_Only:ALPS-1U
- removed SW24: 8, Alps_Only:ALPS-1U
- removed SW25: 9, Alps_Only:ALPS-1U
- removed SW26: 0, Alps_Only:ALPS-1U
- removed SW27: -, Alps_Only:ALPS-1U
- removed SW28: =, Alps_Only:ALPS-1U
- removed SW29: Backspace, Alps_Only:ALPS-1.75U
- removed SW3: F1, Alps_Only:ALPS-1U
- removed SW30: insert, Alps_Only:ALPS-1U
- removed SW31: home, Alps_Only:ALPS-1U
- removed SW32: NUM_lock, Alps_Only:ALPS-1U
- removed SW33: num_/, Alps_Only:ALPS-1U
- removed SW34: num_*, Alps_Only:ALPS-1U
- removed SW35: num_-, Alps_Only:ALPS-1U
- removed SW36: G2, Alps_Only:ALPS-1U
- removed SW37: TAB, Alps_Only:ALPS-1.5U
- removed SW38: Q, Alps_Only:ALPS-1U
- removed SW39: W, Alps_Only:ALPS-1U
- removed SW4: F2, Alps_Only:ALPS-1U
- removed SW40: E, Alps_Only:ALPS-1U
- removed SW41: R, Alps_Only:ALPS-1U
- removed SW42: T, Alps_Only:ALPS-1U
- removed SW43: Y, Alps_Only:ALPS-1U
- removed SW44: U, Alps_Only:ALPS-1U
- removed SW45: I, Alps_Only:ALPS-1U
- removed SW46: O, Alps_Only:ALPS-1U
- removed SW47: P, Alps_Only:ALPS-1U
- removed SW48: [, Alps_Only:ALPS-1U
- removed SW49: ], Alps_Only:ALPS-1U
- removed SW5: F3, Alps_Only:ALPS-1U
- removed SW50: \, Alps_Only:ALPS-1.5U
- removed SW51: END, Alps_Only:ALPS-1U
- removed SW52: PGUP, Alps_Only:ALPS-1U
- removed SW53: num_7, Alps_Only:ALPS-1U
- removed SW54: num_8, Alps_Only:ALPS-1U
- removed SW55: num_9, Alps_Only:ALPS-1U
- removed SW56: G3, Alps_Only:ALPS-1U
- removed SW57: CAP_LOCK, Alps_Only:ALPS-1.75U
- removed SW58: A, Alps_Only:ALPS-1U
- removed SW59: S, Alps_Only:ALPS-1U
- removed SW6: F4, Alps_Only:ALPS-1U
- removed SW60: D, Alps_Only:ALPS-1U
- removed SW61: F, Alps_Only:ALPS-1U
- removed SW62: G, Alps_Only:ALPS-1U
- removed SW63: H, Alps_Only:ALPS-1U
- removed SW64: J, Alps_Only:ALPS-1U
- removed SW65: K, Alps_Only:ALPS-1U
- removed SW66: L, Alps_Only:ALPS-1U
- removed SW67: ;, Alps_Only:ALPS-1U
- removed SW68: ', Alps_Only:ALPS-1U
- removed SW69: ENTER, Alps_Only:ALPS-2.25U
- removed SW7: F5, Alps_Only:ALPS-1U
- removed SW70: DELETE, Alps_Only:ALPS-1U
- removed SW71: PGDN, Alps_Only:ALPS-1U
- removed SW72: num_4, Alps_Only:ALPS-1U
- removed SW73: num_5, Alps_Only:ALPS-1U
- removed SW74: num_6, Alps_Only:ALPS-1U
- removed SW75: num_+, Alps_Only:ALPS-2U
- removed SW76: G4, Alps_Only:ALPS-1U
- removed SW77: LSHIFT, Alps_Only:ALPS-2.25U
- removed SW78: Z, Alps_Only:ALPS-1U
- removed SW79: X, Alps_Only:ALPS-1U
- removed SW8: F6, Alps_Only:ALPS-1U
- removed SW80: C, Alps_Only:ALPS-1U
- removed SW81: V, Alps_Only:ALPS-1U
- removed SW82: B, Alps_Only:ALPS-1U
- removed SW83: N, Alps_Only:ALPS-1U
- removed SW84: M, Alps_Only:ALPS-1U
- removed SW85: ,, Alps_Only:ALPS-1U
- removed SW86: ., Alps_Only:ALPS-1U
- removed SW87: /, Alps_Only:ALPS-1U
- removed SW88: RSHIFT, Alps_Only:ALPS-2.5U
- removed SW89: arrow_UP, Alps_Only:ALPS-1U
- removed SW9: F7, Alps_Only:ALPS-1U
- removed SW90: num_1, Alps_Only:ALPS-1U
- removed SW91: num_2, Alps_Only:ALPS-1U
- removed SW92: num_3, Alps_Only:ALPS-1U
- removed SW93: LCRTL, Alps_Only:ALPS-1.25U
- removed SW94: WIN, Alps_Only:ALPS-1.25U
- removed SW95: LALT, Alps_Only:ALPS-1.25U
- removed SW96: SPACE, Alps_Only:ALPS-6.25U
- removed SW97: RALT, Alps_Only:ALPS-1.25U
- removed SW98: MENU, Alps_Only:ALPS-1.25U
- removed SW99: RCRTL, Alps_Only:ALPS-1.25U
- removed USB1: HRO-TYPE-C-31-M-12, Type-C.pretty-master:HRO-TYPE-C-31-M-12-HandSoldering
- added C1: 0.1u, Capacitor_SMD:C_0402_1005Metric, B.Cu at (154.8, 108.7)
- added C10: 100n, Capacitor_SMD:C_0402_1005Metric, B.Cu at (156.4, 118.3)
- added C11: 100n, Capacitor_SMD:C_0402_1005Metric, B.Cu at (148.9, 125.6)
- added C12: 100n, Capacitor_SMD:C_0402_1005Metric, B.Cu at (143.4, 118.7)
- added C13: 100n, Capacitor_SMD:C_0402_1005Metric, B.Cu at (155.6, 114.1)
- added C14: 100n, Capacitor_SMD:C_0402_1005Metric, B.Cu at (148.9, 108.0)
- added C15: 100n, Capacitor_SMD:C_0402_1005Metric, B.Cu at (146.4, 111.5)
- added C16: 100n, Capacitor_SMD:C_0402_1005Metric, B.Cu at (147.4, 111.5)
- added J1: Conn_01x05, Connector_PinHeader_2.54mm:PinHeader_1x05_P2.54mm_Vertical, B.Cu at (146.4, 131.0)
- added J2: USB_C_Receptacle_USB2.0_16P, Connector_USB:USB_C_Receptacle_HRO_TYPE-C-31-M-12, B.Cu at (69.1, 16.7)
- added J3: Conn_01x04, Connector_JST:JST_SH_SM04B-SRSS-TB_1x04-1MP_P1.00mm_Horizontal, B.Cu at (69.8, 33.3)
- added MX10: 1u, PCM_marbastlib-mx:SW_MX_HS_CPG151101S11_1u, B.Cu at (257.2, 23.8)
- added MX11: 1u, PCM_marbastlib-mx:SW_MX_HS_CPG151101S11_1u, B.Cu at (276.2, 23.8)
- added MX12: 1u, PCM_marbastlib-mx:SW_MX_HS_CPG151101S11_1u, B.Cu at (295.3, 23.8)
- added MX13: 1u, PCM_marbastlib-mx:SW_MX_HS_CPG151101S11_1u, B.Cu at (314.3, 23.8)
- added MX14: 1u, PCM_marbastlib-mx:SW_MX_HS_CPG151101S11_1u, B.Cu at (28.6, 47.6)
- added MX15: 1.25u, PCM_marbastlib-mx:SW_MX_HS_CPG151101S11_1.25u, B.Cu at (54.8, 47.6)
- added MX16: 1u, PCM_marbastlib-mx:SW_MX_HS_CPG151101S11_1u, B.Cu at (76.2, 47.6)
- added MX17: 1u, PCM_marbastlib-mx:SW_MX_HS_CPG151101S11_1u, B.Cu at (95.2, 47.6)
- added MX18: 1u, PCM_marbastlib-mx:SW_MX_HS_CPG151101S11_1u, B.Cu at (114.3, 47.6)
- added MX19: 1u, PCM_marbastlib-mx:SW_MX_HS_CPG151101S11_1u, B.Cu at (133.3, 47.6)
- added MX2: 1u, PCM_marbastlib-mx:SW_MX_HS_CPG151101S11_1u, B.Cu at (85.7, 23.8)
- added MX20: 1u, PCM_marbastlib-mx:SW_MX_HS_CPG151101S11_1u, B.Cu at (152.4, 47.6)
- added MX21: 1u, PCM_marbastlib-mx:SW_MX_HS_CPG151101S11_1u, B.Cu at (171.4, 47.6)
- added MX22: 1u, PCM_marbastlib-mx:SW_MX_HS_CPG151101S11_1u, B.Cu at (190.5, 47.6)
- added MX23: 1u, PCM_marbastlib-mx:SW_MX_HS_CPG151101S11_1u, B.Cu at (209.6, 47.6)
- added MX24: 1u, PCM_marbastlib-mx:SW_MX_HS_CPG151101S11_1u, B.Cu at (228.6, 47.6)
- added MX25: 1u, PCM_marbastlib-mx:SW_MX_HS_CPG151101S11_1u, B.Cu at (247.7, 47.6)
- added MX26: 1u, PCM_marbastlib-mx:SW_MX_HS_CPG151101S11_1u, B.Cu at (266.7, 47.6)
- added MX27: 1u, PCM_marbastlib-mx:SW_MX_HS_CPG151101S11_1u, B.Cu at (285.8, 47.6)
- added MX28: 1.75u, PCM_marbastlib-mx:SW_MX_HS_CPG151101S11_1.75u, B.Cu at (311.9, 47.6)
- added MX29: 1u, PCM_marbastlib-mx:SW_MX_HS_CPG151101S11_1u, B.Cu at (342.9, 38.1)
- added MX3: 1u, PCM_marbastlib-mx:SW_MX_HS_CPG151101S11_1u, B.Cu at (104.8, 23.8)
- added MX30: 1u, PCM_marbastlib-mx:SW_MX_HS_CPG151101S11_1u, B.Cu at (361.9, 38.1)
- added MX31: 1u, PCM_marbastlib-mx:SW_MX_HS_CPG151101S11_1u, B.Cu at (28.6, 66.7)
- added MX32: 1.5u, PCM_marbastlib-mx:SW_MX_HS_CPG151101S11_1.5u, B.Cu at (57.1, 66.7)
- added MX33: 1u, PCM_marbastlib-mx:SW_MX_HS_CPG151101S11_1u, B.Cu at (81.0, 66.7)
- added MX34: 1u, PCM_marbastlib-mx:SW_MX_HS_CPG151101S11_1u, B.Cu at (100.0, 66.7)
- added MX35: 1u, PCM_marbastlib-mx:SW_MX_HS_CPG151101S11_1u, B.Cu at (119.1, 66.7)
- added MX36: 1u, PCM_marbastlib-mx:SW_MX_HS_CPG151101S11_1u, B.Cu at (138.1, 66.7)
- added MX37: 1u, PCM_marbastlib-mx:SW_MX_HS_CPG151101S11_1u, B.Cu at (157.2, 66.7)
- added MX38: 1u, PCM_marbastlib-mx:SW_MX_HS_CPG151101S11_1u, B.Cu at (176.2, 66.7)
- added MX39: 1u, PCM_marbastlib-mx:SW_MX_HS_CPG151101S11_1u, B.Cu at (195.3, 66.7)
- added MX4: 1u, PCM_marbastlib-mx:SW_MX_HS_CPG151101S11_1u, B.Cu at (123.8, 23.8)
- added MX40: 1u, PCM_marbastlib-mx:SW_MX_HS_CPG151101S11_1u, B.Cu at (214.3, 66.7)
- added MX41: 1u, PCM_marbastlib-mx:SW_MX_HS_CPG151101S11_1u, B.Cu at (233.4, 66.7)
- added MX42: 1u, PCM_marbastlib-mx:SW_MX_HS_CPG151101S11_1u, B.Cu at (252.4, 66.7)
- added MX43: 1u, PCM_marbastlib-mx:SW_MX_HS_CPG151101S11_1u, B.Cu at (271.5, 66.7)
- added MX44: 1u, PCM_marbastlib-mx:SW_MX_HS_CPG151101S11_1u, B.Cu at (290.5, 66.7)
- added MX45: 1.5u, PCM_marbastlib-mx:SW_MX_HS_CPG151101S11_1.5u, B.Cu at (314.3, 66.7)
- added MX46: 1u, PCM_marbastlib-mx:SW_MX_HS_CPG151101S11_1u, B.Cu at (342.9, 57.1)
- added MX47: 1u, PCM_marbastlib-mx:SW_MX_HS_CPG151101S11_1u, B.Cu at (361.9, 57.1)
- added MX48: 1u, PCM_marbastlib-mx:SW_MX_HS_CPG151101S11_1u, B.Cu at (28.6, 85.7)
- added MX49: 1.75u, PCM_marbastlib-mx:SW_MX_HS_CPG151101S11_1.75u, B.Cu at (59.5, 85.7)
- added MX5: 1u, PCM_marbastlib-mx:SW_MX_HS_CPG151101S11_1u, B.Cu at (142.9, 23.8)
- added MX50: 1u, PCM_marbastlib-mx:SW_MX_HS_CPG151101S11_1u, B.Cu at (85.7, 85.7)
- added MX51: 1u, PCM_marbastlib-mx:SW_MX_HS_CPG151101S11_1u, B.Cu at (104.8, 85.7)
- added MX52: 1u, PCM_marbastlib-mx:SW_MX_HS_CPG151101S11_1u, B.Cu at (123.8, 85.7)
- added MX53: 1u, PCM_marbastlib-mx:SW_MX_HS_CPG151101S11_1u, B.Cu at (142.9, 85.7)
- added MX54: 1u, PCM_marbastlib-mx:SW_MX_HS_CPG151101S11_1u, B.Cu at (161.9, 85.7)
- added MX55: 1u, PCM_marbastlib-mx:SW_MX_HS_CPG151101S11_1u, B.Cu at (181.0, 85.7)
- added MX56: 1u, PCM_marbastlib-mx:SW_MX_HS_CPG151101S11_1u, B.Cu at (200.0, 85.7)
- added MX57: 1u, PCM_marbastlib-mx:SW_MX_HS_CPG151101S11_1u, B.Cu at (219.1, 85.7)
- added MX58: 1u, PCM_marbastlib-mx:SW_MX_HS_CPG151101S11_1u, B.Cu at (238.1, 85.7)
- added MX59: 1u, PCM_marbastlib-mx:SW_MX_HS_CPG151101S11_1u, B.Cu at (257.2, 85.7)
- added MX6: 1u, PCM_marbastlib-mx:SW_MX_HS_CPG151101S11_1u, B.Cu at (171.4, 23.8)
- added MX60: 1u, PCM_marbastlib-mx:SW_MX_HS_CPG151101S11_1u, B.Cu at (276.2, 85.7)
- added MX61: 1u, PCM_marbastlib-mx:SW_MX_HS_CPG151101S11_1u, B.Cu at (307.2, 85.7)
- added MX62: 1u, PCM_marbastlib-mx:SW_MX_HS_CPG151101S11_1u, B.Cu at (342.9, 76.2)
- added MX63: 1u, PCM_marbastlib-mx:SW_MX_HS_CPG151101S11_1u, B.Cu at (361.9, 76.2)
- added MX64: 1u, PCM_marbastlib-mx:SW_MX_HS_CPG151101S11_1u, B.Cu at (28.6, 104.8)
- added MX65: 1u, PCM_marbastlib-mx:SW_MX_HS_CPG151101S11_1u, B.Cu at (64.3, 104.8)
- added MX66: 1u, PCM_marbastlib-mx:SW_MX_HS_CPG151101S11_1u, B.Cu at (95.2, 104.8)
- added MX67: 1u, PCM_marbastlib-mx:SW_MX_HS_CPG151101S11_1u, B.Cu at (114.3, 104.8)
- added MX68: 1u, PCM_marbastlib-mx:SW_MX_HS_CPG151101S11_1u, B.Cu at (133.3, 104.8)
- added MX69: 1u, PCM_marbastlib-mx:SW_MX_HS_CPG151101S11_1u, B.Cu at (152.4, 104.8)
- added MX7: 1u, PCM_marbastlib-mx:SW_MX_HS_CPG151101S11_1u, B.Cu at (190.5, 23.8)
- added MX70: 1u, PCM_marbastlib-mx:SW_MX_HS_CPG151101S11_1u, B.Cu at (171.4, 104.8)
- added MX71: 1u, PCM_marbastlib-mx:SW_MX_HS_CPG151101S11_1u, B.Cu at (190.5, 104.8)
- added MX72: 1u, PCM_marbastlib-mx:SW_MX_HS_CPG151101S11_1u, B.Cu at (209.6, 104.8)
- added MX73: 1u, PCM_marbastlib-mx:SW_MX_HS_CPG151101S11_1u, B.Cu at (228.6, 104.8)
- added MX74: 1u, PCM_marbastlib-mx:SW_MX_HS_CPG151101S11_1u, B.Cu at (247.7, 104.8)
- added MX75: 1u, PCM_marbastlib-mx:SW_MX_HS_CPG151101S11_1u, B.Cu at (266.7, 104.8)
- added MX76: 1u, PCM_marbastlib-mx:SW_MX_HS_CPG151101S11_1u, B.Cu at (302.4, 104.8)
- added MX77: 1u, PCM_marbastlib-mx:SW_MX_HS_CPG151101S11_1u, B.Cu at (342.9, 104.8)
- added MX78: 1.25u, PCM_marbastlib-mx:SW_MX_HS_CPG151101S11_1.25u, B.Cu at (54.8, 123.8)
- added MX79: 1.25u, PCM_marbastlib-mx:SW_MX_HS_CPG151101S11_1.25u, B.Cu at (78.6, 123.8)
- added MX8: 1u, PCM_marbastlib-mx:SW_MX_HS_CPG151101S11_1u, B.Cu at (209.6, 23.8)
- added MX80: 1.25u, PCM_marbastlib-mx:SW_MX_HS_CPG151101S11_1.25u, B.Cu at (102.4, 123.8)
- added MX81: 1u, PCM_marbastlib-mx:SW_MX_HS_CPG151101S11_1u, B.Cu at (173.8, 123.8)
- added MX82: 1.25u, PCM_marbastlib-mx:SW_MX_HS_CPG151101S11_1.25u, B.Cu at (245.3, 123.8)
- added MX83: 1.25u, PCM_marbastlib-mx:SW_MX_HS_CPG151101S11_1.25u, B.Cu at (269.1, 123.8)
- added MX84: 1.5u, PCM_marbastlib-mx:SW_MX_HS_CPG151101S11_1.5u, B.Cu at (295.3, 123.8)
- added MX85: 1u, PCM_marbastlib-mx:SW_MX_HS_CPG151101S11_1u, B.Cu at (323.9, 123.8)
- added MX86: 1u, PCM_marbastlib-mx:SW_MX_HS_CPG151101S11_1u, B.Cu at (342.9, 123.8)
- added MX87: 1u, PCM_marbastlib-mx:SW_MX_HS_CPG151101S11_1u, B.Cu at (361.9, 123.8)
- added MX9: 1u, PCM_marbastlib-mx:SW_MX_HS_CPG151101S11_1u, B.Cu at (228.6, 23.8)
- added Mx1: 1u, PCM_marbastlib-mx:SW_MX_HS_CPG151101S11_1u, B.Cu at (52.4, 23.8)
- added S1: MX_stab, PCM_marbastlib-mx:STAB_MX_P_6.25u, F.Cu at (173.6, 123.5)
- added S2: MX_stab, PCM_marbastlib-mx:STAB_MX_P_2.25u, F.Cu at (307.2, 85.7)
- added S3: MX_stab, PCM_marbastlib-mx:STAB_MX_P_2.25u, F.Cu at (64.3, 104.8)
- added S4: MX_stab, PCM_marbastlib-mx:STAB_MX_P_2.25u, F.Cu at (302.4, 104.8)
- added U3: RP2040, Package_DFN_QFN:QFN-56-1EP_7x7mm_P0.4mm_EP3.2x3.2mm, B.Cu at (150.0, 117.5)
- added U5: SRV05-4, PCM_marbastlib-various:SOT-23-6-routable, B.Cu at (69.5, 26.8)
- C2, C3, C9: footprint Capacitor_SMD:C_0805_2012Metric_Pad1.18x1.45mm_HandSolder -> Capacitor_SMD:C_0402_1005Metric
- C4, C5: value 0.1u -> 22p; footprint Capacitor_SMD:C_0805_2012Metric_Pad1.18x1.45mm_HandSolder -> Capacitor_SMD:C_0402_1005Metric
- C6: value 0.1u -> 1u; footprint Capacitor_SMD:C_0805_2012Metric_Pad1.18x1.45mm_HandSolder -> Capacitor_SMD:C_0402_1005Metric
- C7: value 0.1u -> 100n; footprint Capacitor_SMD:C_0805_2012Metric_Pad1.18x1.45mm_HandSolder -> Capacitor_SMD:C_0402_1005Metric
- C8: footprint Capacitor_SMD:C_0805_2012Metric_Pad1.18x1.45mm_HandSolder -> Capacitor_SMD:C_0603_1608Metric
- D1, D10, D11, D12, D13, D14, D15, D16, D17, D18, D19, D2, D20, D21, D22, D23, D24, D25, D26, D27, D28, D29, D3, D30, D31, D32, D33, D34, D35, D36, D37, D38, D39, D4, D40, D41, D42, D43, D44, D45, D46, D47, D48, D49, D5, D50, D51, D52, D53, D54, D55, D56, D57, D58, D59, D6, D60, D61, D62, D63, D64, D65, D66, D67, D68, D69, D7, D70, D71, D72, D73, D74, D75, D76, D77, D78, D79, D8, D80, D81, D82, D83, D84, D85, D86, D87, D9: footprint Diode_SMD:D_0201_0603Metric_Pad0.64x0.40mm_HandSolder -> Diode_SMD:D_SOD-123
- F1: value 500m -> Fuse_Small; footprint Fuse:Fuse_1206_3216Metric_Pad1.42x1.75mm_HandSolder -> Fuse:Fuse_1206_3216Metric
- R1: value 1k -> 5.1k; footprint Resistor_SMD:R_0805_2012Metric_Pad1.20x1.40mm_HandSolder -> Resistor_SMD:R_0402_1005Metric
- R2: value 10k -> 5.1k; footprint Resistor_SMD:R_0805_2012Metric_Pad1.20x1.40mm_HandSolder -> Resistor_SMD:R_0402_1005Metric
- R3, R4: value 22 -> 5.1k; footprint Resistor_SMD:R_0805_2012Metric_Pad1.20x1.40mm_HandSolder -> Resistor_SMD:R_0402_1005Metric
- R5: value 5.1k -> 1k; footprint Resistor_SMD:R_0805_2012Metric_Pad1.20x1.40mm_HandSolder -> Resistor_SMD:R_0402_1005Metric
- R6: footprint Resistor_SMD:R_0805_2012Metric_Pad1.20x1.40mm_HandSolder -> Resistor_SMD:R_0402_1005Metric
- R7: value 10k -> 1k; footprint Resistor_SMD:R_0805_2012Metric_Pad1.20x1.40mm_HandSolder -> Resistor_SMD:R_0402_1005Metric
- R8: value 2k -> 5.1k; footprint Resistor_SMD:R_0805_2012Metric_Pad1.20x1.40mm_HandSolder -> Resistor_SMD:R_0402_1005Metric
- R9: value 1k -> 5.1k; footprint Resistor_SMD:R_0805_2012Metric_Pad1.20x1.40mm_HandSolder -> Resistor_SMD:R_0402_1005Metric; moved to B.Cu
- SW1: footprint Button_Switch_SMD:SW_SPST_SKQG_WithStem -> Button_Switch_SMD:SW_Push_1P1T_XKB_TS-1187A
- SW2: value esc -> Switch; footprint Alps_Only:ALPS-1U -> Button_Switch_SMD:SW_Push_1P1T_XKB_TS-1187A; moved to B.Cu
- U1: value PRTR5V0U2X -> XC6206PxxxMR; footprint random-keyboard-parts.pretty-master:SOT143B -> Package_TO_SOT_SMD:SOT-23-3
- U2: value AT90USB646-A -> W25Q128JVS; footprint Package_QFP:TQFP-64_14x14mm_P0.8mm -> Package_SO:SOIC-8_5.23x5.23mm_P1.27mm
- Y1: value Crystal_GND24_Small -> Crystal_GND24; footprint Crystal:Crystal_SMD_3225-4Pin_3.2x2.5mm_HandSoldering -> Crystal:Crystal_SMD_3225-4Pin_3.2x2.5mm
- moved D31 360.7 mm to (31.8, 67.5)
- moved D32 351.1 mm to (60.3, 67.5)
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Connections:
- C2 pad 1: XTAL1 -> +5V
- C3 pad 1: XTAL2 -> +3V3
- C4 pad 1: +5V -> X IN
- C5 pad 1: +5V -> Net-(C5-Pad1)
- C6 pad 1: +5V -> +1V1
- C7 pad 1: +5V -> +1V1
- C8 pad 1: +5V -> +3V3
- C9 pad 1: Net-(U2-UCAP) -> +3V3
- D31 pad 1: row 1 -> row 2
- D32 pad 1: row 1 -> row 2
- D33 pad 1: row 1 -> row 2
- D34 pad 1: row 1 -> row 2
- D45 pad 2: /matrix/2 -> Net-(D45-A)
- D48 pad 1: row 2 -> row 3
- D49 pad 1: row 2 -> row 3
- D50 pad 1: row 2 -> row 3
- D51 pad 1: row 2 -> row 3
- D52 pad 1: row 2 -> row 3
- D53 pad 1: row 2 -> row 3
- D54 pad 1: row 2 -> row 3
- D64 pad 1: row 3 -> row 4
- D65 pad 1: row 3 -> row 4
- D66 pad 1: row 3 -> row 4
- D67 pad 1: row 3 -> row 4
- D68 pad 1: row 3 -> row 4
- D69 pad 1: row 3 -> row 4
- D70 pad 1: row 3 -> row 4
- D71 pad 1: row 3 -> row 4
- D72 pad 1: row 3 -> row 4
- D73 pad 1: row 3 -> row 4
- D74 pad 1: row 3 -> row 4
- D78 pad 1: row 4 -> row 5
- D79 pad 1: row 4 -> row 5
- D80 pad 1: row 4 -> row 5
- D81 pad 1: row 4 -> row 5
- D82 pad 1: row 4 -> row 5
- D83 pad 1: row 4 -> row 5
- D84 pad 1: row 4 -> row 5
- D85 pad 1: row 4 -> row 5
- D86 pad 1: row 4 -> row 5
- D87 pad 1: row 4 -> row 5
- F1 pad 1: /VCC -> VBUS
- R1 pad 1: LED -> GND
- R1 pad 2: Net-(Q1-B) -> Net-(J2-CC1)
- R2 pad 1: RESET -> Net-(J2-CC2)
- R2 pad 2: +5V -> GND
- R3 pad 1: Net-(U1-IO2) -> +3V3
- R3 pad 2: D- -> RESET
- R4 pad 1: Net-(U1-IO1) -> +3V3
- R4 pad 2: D+ -> Net-(R4-Pad2)
- R5 pad 1: Net-(USB1-CC1) -> Net-(C5-Pad1)
- R5 pad 2: GND -> X OUT
- R6 pad 1: Net-(USB1-CC2) -> Q SEL
- R6 pad 2: GND -> Net-(R4-Pad2)
- R7 pad 1: GND -> Q SEL
- R7 pad 2: Net-(U2-PE2/~{HWB}) -> Net-(R7-Pad2)
- R8 pad 2: Net-(Q1-B) -> D+
- R9 pad 1: Net-(Q1-C) -> D-
- SW2 pad 1: col 1 -> GND
- SW2 pad 2: Net-(D1-A) -> Net-(R7-Pad2)
- U1 pad 2: Net-(U1-IO1) -> +3V3
- U1 pad 3: Net-(U1-IO2) -> +5V
- U2 pad 1: unconnected-(U2-PE6-Pad1) -> Q SEL
- U2 pad 2: unconnected-(U2-PE7-Pad2) -> Q 01
- U2 pad 3: +5V -> Q 02
- U2 pad 4: D- -> GND
- U2 pad 5: D+ -> Q 00
- U2 pad 6: GND -> Q CLK
- U2 pad 7: Net-(U2-UCAP) -> Q 03
- U2 pad 8: +5V -> +3V3
- Y1 pad 1: XTAL1 -> Net-(C5-Pad1)
- Y1 pad 3: XTAL2 -> X IN
Routing:
- net col 20: track 317.8 -> 0.00 mm, vias 1 -> 0
- net col 19: track 299.5 -> 0.00 mm, vias 1 -> 0
- net col 18: track 281.1 -> 0.00 mm, vias 1 -> 0
- net col 17: track 274.2 -> 0.00 mm, vias 1 -> 0
- net D+: track 8.78 -> 171.6 mm
- net D-: track 7.54 -> 168.4 mm
- net +3V3: track 0.00 -> 135.8 mm, vias 0 -> 4
- net GND: track 40.8 -> 172.6 mm, vias 0 -> 31
- net +5V: track 18.8 -> 141.0 mm
- net col 11: track 140.8 -> 208.1 mm, vias 3 -> 2
- net row 5: track 396.9 -> 330.4 mm, vias 3 -> 11
- net col 13: track 198.5 -> 256.0 mm, vias 1 -> 2
- net col 9: track 105.0 -> 162.0 mm, vias 1 -> 2
- net col 4: track 187.6 -> 135.1 mm, vias 1 -> 2
- net col 3: track 214.5 -> 162.4 mm, vias 4 -> 2
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- added copper zone on B.Cu, net GND
- added copper zone on F.Cu, net GND
Other:
- board size 438.2 x 123 mm -> 352.1 x 121.7 mm
- board text added: "JLCJLCJLCJLC"
