File: test2.kicad_sch (KiCad schematic)
At the start: 23 parts, among them J1 AVR-ISP-6, SW1 Reset, U1 PRTR5V0U2X, U2 ATmega32U4-A, U3 STM32F401CCUx, Y1 Crystal_GND24_Small

Commit message: project resumed
Parts:
- removed C9: 1u, symbol Device:C_Small
- removed F1: 500m, symbol Device:Polyfuse_Small
- removed J1: AVR-ISP-6, symbol Connector:AVR-ISP-6
- removed SW1: Reset, symbol Switch:SW_Push
- removed U1: PRTR5V0U2X, symbol random-keyboard-parts:PRTR5V0U2X
- removed U2: ATmega32U4-A, Package_QFP:TQFP-44_10x10mm_P0.8mm, symbol MCU_Microchip_ATmega:ATmega32U4-A
- removed U3: STM32F401CCUx, Package_DFN_QFN:QFN-48-1EP_7x7mm_P0.5mm_EP5.6x5.6mm, symbol MCU_ST_STM32F4:STM32F401CCUx
- removed USB1: HRO-TYPE-C-31-M-12, symbol Type-C:HRO-TYPE-C-31-M-12
- removed Y1: Crystal_GND24_Small, symbol Device:Crystal_GND24_Small
- added C4, C5: 22p, Capacitor_SMD:C_0402_1005Metric, symbol Device:C_Small
- added C6: 1u, Capacitor_SMD:C_0402_1005Metric, symbol Device:C_Small
- added C7: 100n, Capacitor_SMD:C_0402_1005Metric, symbol Device:C_Small
- added F1: Fuse_Small, symbol Device:Fuse_Small
- added J1: Conn_01x05, Connector_USB:USB_C_Receptacle_HRO_TYPE-C-31-M-12, symbol Connector_Generic:Conn_01x05
- added J2: USB_C_Receptacle_USB2.0_16P, Connector_JST:JST_SH_SM04B-SRSS-TB_1x04-1MP_P1.00mm_Horizontal, symbol Connector:USB_C_Receptacle_USB2.0_16P
- added J3: Conn_01x04, Connector_PinHeader_2.54mm:PinHeader_1x05_P2.54mm_Vertical, symbol Connector_Generic:Conn_01x04
- added R7: 1k, Resistor_SMD:R_0805_2012Metric_Pad1.20x1.40mm_HandSolder, symbol Device:R_Small
- added R8, R9: 5.1k, Resistor_SMD:R_0402_1005Metric, symbol Device:R_Small
- added SW1, SW2: Switch, Button_Switch_SMD:SW_Push_1P1T_XKB_TS-1187A, symbol ScottoKeebs:Placeholder_Switch
- added U1: XC6206PxxxMR, Package_TO_SOT_SMD:SOT-23-3, symbol Regulator_Linear:XC6206PxxxMR
- added U2: W25Q128JVS, Package_SO:SOIC-8_5.23x5.23mm_P1.27mm, symbol Memory_Flash:W25Q128JVS
- added U3: RP2040, Package_DFN_QFN:QFN-56-1EP_7x7mm_P0.4mm_EP3.2x3.2mm, symbol MCU_RaspberryPi:RP2040
- added U4: SRV05-4, Package_TO_SOT_SMD:SOT-23-3, symbol PCM_marbastlib-various:SRV05-4
- added Y1: Crystal_GND24, Crystal:Crystal_SMD_3225-4Pin_3.2x2.5mm, symbol Device:Crystal_GND24
- C1: value 1u -> 0.1u; footprint (none) -> Capacitor_SMD:C_0402_1005Metric
- C10: renamed from C6; value 0.1u -> 100n; footprint (none) -> Capacitor_SMD:C_0402_1005Metric
- C11: renamed from C7; value 0.1u -> 100n; footprint (none) -> Capacitor_SMD:C_0402_1005Metric
- C12: renamed from C8; value 0.1u -> 100n; footprint (none) -> Capacitor_SMD:C_0402_1005Metric
- C2, C3: footprint (none) -> Capacitor_SMD:C_0402_1005Metric
- C8: renamed from C4; value 0.1u -> 10u; footprint (none) -> Capacitor_SMD:C_0603_1608Metric
- C9: renamed from C5; value 0.1u -> 1u; footprint (none) -> Capacitor_SMD:C_0402_1005Metric
- R1, R2: value 10k -> 5.1k; footprint (none) -> Resistor_SMD:R_0402_1005Metric
- R3, R4: value 22 -> 5.1k; footprint (none) -> Resistor_SMD:R_0805_2012Metric_Pad1.20x1.40mm_HandSolder
- R5: value 5.1k -> 1k; footprint (none) -> Resistor_SMD:R_0402_1005Metric
- R6: footprint (none) -> Resistor_SMD:R_0402_1005Metric
Connections:
- net XTAL1 is gone; now on net +5V: C2.1
- net XTAL2 is gone; now on net +3V3: C3.1
- net +5V: now also F1.2, J3.1 (Pin_1), U1.3 (VI), U4.5 (VP); no longer C10.1, C11.1, C12.1, C8.1, C9.1, R2.2
- net D+: now also J2.A6 (D+), J2.B6 (D+), J3.3 (Pin_3), R8.2, U4.6 (IO4); no longer R4.2
- net D-: now also J2.A7 (D-), J2.B7 (D-), J3.2 (Pin_2), R9.1, U4.1 (IO1); no longer R3.2
- net GND: now also R2.2, C4.2, C5.2, C6.2, C7.2, J1.3 (Pin_3), J2.A1 (GND), J2.A12 (GND), J2.B1 (GND), J2.B12 (GND), J2.S1 (SHIELD), J3.4 (Pin_4), SW1.1, SW2.1, U1.1 (GND), U2.4 (GND), U3.19 (TESTEN), U3.57 (GND), U4.2 (VN), Y1.2, Y1.4; no longer R5.2, R6.2
- net RESET: now also R3.2, J1.1 (Pin_1), SW1.2, U3.26 (RUN); no longer R2.1
- net +3V3: now reaches R4.1
- net +3V3: now also C1.1, C10.1, C11.1, C12.1, C8.1, C9.1, R3.1, J1.2 (Pin_2), U1.2 (VO), U2.8 (VCC), U3.1 (IOVDD), U3.10 (IOVDD), U3.22 (IOVDD), U3.33 (IOVDD), U3.42 (IOVDD), U3.43 (ADC_AVDD), U3.44 (VREG_IN), U3.48 (USB_VDD), U3.49 (IOVDD)
- net Q SEL: now reaches R6.1
- net Q SEL: now also R7.1, U2.1 (~{CS}), U3.56 (QSPI_SS)
- net at R1.2: now also J2.A5 (CC1)
- net at R5.1: now also C5.1, Y1.1
- new net: R8.1, U3.47 (USB_DP)
- new net: R7.2, SW2.2
- new net: R9.2, U3.46 (USB_DM)
- new net: R4.2, R6.2
- new net: J2.B5 (CC2), R2.1
- new net +1V1: C6.1, C7.1, U3.23 (DVDD), U3.45 (VREG_VOUT), U3.50 (DVDD)
- new net Q 00: U2.5 (DI(IO0)), U3.53 (QSPI_SD0)
- new net Q 01: U2.2 (DO(IO1)), U3.55 (QSPI_SD1)
- new net Q 02: U2.3 (IO2), U3.54 (QSPI_SD2)
- new net Q 03: U2.7 (IO3), U3.51 (QSPI_SD3)
- new net Q CLK: U2.6 (CLK), U3.52 (QSPI_SCLK)
- new net SWC: J1.4 (Pin_4), U3.24 (SWCLK)
- new net SWD: J1.5 (Pin_5), U3.25 (SWD)
- new net VBUS: F1.1, J2.A4 (VBUS), J2.A9 (VBUS), J2.B4 (VBUS), J2.B9 (VBUS)
- new net X IN: C4.1, U3.20 (XIN), Y1.3
- new net X OUT: R5.2, U3.21 (XOUT)
- no-connect marks 6 -> 4
Other:
- added sheet LED_sheet (LED.kicad_sch)
- moved on the sheet: C10, C11, C12, C8, C9

Commit message: Finalization of 89 key
Changed 104 keys to 89, removed LEDs, created files needed for production.
Parts:
- removed U4: SRV05-4, Package_TO_SOT_SMD:SOT-23-3, symbol PCM_marbastlib-various:SRV05-4
- added C13, C14, C15, C16: 100n, Capacitor_SMD:C_0402_1005Metric, symbol Device:C_Small
- added U5: SRV05-4, PCM_marbastlib-various:SOT-23-6-routable, symbol PCM_marbastlib-various:SRV05-4
- F1: footprint (none) -> Fuse:Fuse_1206_3216Metric
- J1: footprint Connector_USB:USB_C_Receptacle_HRO_TYPE-C-31-M-12 -> Connector_PinHeader_2.54mm:PinHeader_1x05_P2.54mm_Vertical
- J2: footprint Connector_JST:JST_SH_SM04B-SRSS-TB_1x04-1MP_P1.00mm_Horizontal -> Connector_USB:USB_C_Receptacle_HRO_TYPE-C-31-M-12
- J3: footprint Connector_PinHeader_2.54mm:PinHeader_1x05_P2.54mm_Vertical -> Connector_JST:JST_SH_SM04B-SRSS-TB_1x04-1MP_P1.00mm_Horizontal
- R3, R4, R7: footprint Resistor_SMD:R_0805_2012Metric_Pad1.20x1.40mm_HandSolder -> Resistor_SMD:R_0402_1005Metric
Connections:
- net +1V1: now also C16.1
- net +3V3: now also J1.4 (Pin_4), C13.1, C14.1, C15.1; no longer J1.2 (Pin_2)
- net +5V: now also U5.5 (VP)
- net D+: now also U5.1 (IO1)
- net D-: now also U5.6 (IO4)
- net GND: now also J1.5 (Pin_5), C13.2, C14.2, C15.2, C16.2, U5.2 (VN); no longer J1.3 (Pin_3)
- net RESET: now also J1.3 (Pin_3); no longer J1.1 (Pin_1)
- net SWC: now also J1.1 (Pin_1); no longer J1.4 (Pin_4)
- net SWD: now also J1.2 (Pin_2); no longer J1.5 (Pin_5)
- net col 0: now also U3.27 (GPIO16)
- net col 1: now also U3.28 (GPIO17)
- net col 10: now also U3.6 (GPIO4)
- net col 11: now also U3.9 (GPIO7)
- net col 12: now also U3.8 (GPIO6)
- net col 13: now also U3.11 (GPIO8)
- net col 14: now also U3.7 (GPIO5)
- net col 15: now also U3.12 (GPIO9)
- net col 16: now also U3.13 (GPIO10)
- net col 2: now also U3.29 (GPIO18)
- net col 3: now also U3.30 (GPIO19)
- net col 4: now also U3.31 (GPIO20)
- net col 5: now also U3.32 (GPIO21)
- net col 6: now also U3.2 (GPIO0)
- net col 7: now also U3.16 (GPIO13)
- net col 8: now also U3.4 (GPIO2)
- net col 9: now also U3.5 (GPIO3)
- net row 0: now also U3.37 (GPIO25)
- net row 1: now also U3.36 (GPIO24)
- net row 2: now also U3.35 (GPIO23)
- net row 3: now also U3.34 (GPIO22)
- net row 4: now also U3.17 (GPIO14)
- net row 5: now also U3.18 (GPIO15)
- no-connect marks 4 -> 8
Other:
- removed sheet LED_sheet
